File: EPS_PDU.kicad_sch (KiCad schematic)
At the start: 150 parts, among them IC1 INA226AIDGSR, IC10 MAX17523ATE+, IC11 LM74700QDBVRQ1, IC12 LM74700QDBVRQ1, IC13 L6982C50DR, IC14 L6982C33DR, IC15 MAX17523ATE+, IC16 LM74700QDBVRQ1, IC17 L6982C33DR, IC18 MAX890LESA+, IC19 LM74700QDBVRQ1, IC2 L6982C33DR, IC20 INA226AIDGSR, IC21 LM74700QDBVRQ1, IC22 LM74700QDBVRQ1, IC23 LM74700QDBVRQ1, IC24 L6982C50DR, IC3 MAX890LESA+, IC4 MAX17523ATE+, IC5 LM74700QDBVRQ1, IC6 LM74700QDBVRQ1, IC7 MAX17523ATE+, IC8 LM74700QDBVRQ1, IC9 MAX17523ATE+, Q1 DMN4035LQ-13, Q10 DMN4035LQ-13, Q2 DMN4035LQ-13, Q3 DMN4035LQ-13, Q4 DMN4035LQ-13, Q5 DMN4035LQ-13, Q6 DMN4035LQ-13, Q7 DMN4035LQ-13, Q8 DMN4035LQ-13, Q9 DMN4035LQ-13

Commit message: UART ic added, SWD pins mapped
Parts:
- renumbered C52 to C10, C7 to C11, C64 to C13, C61 to C14, C58 to C15, C53 to C16, C6 to C17, C54 to C18, C15 to C19, C65 to C20, C62 to C21, C59 to C22, C1 to C23, C57 to C24, C66 to C25, C55 to C26, C63 to C27, C16 to C28, C60 to C29, C56 to C30, C17 to C31, C18 to C32, C25 to C33, C26 to C34, C43 to C35, C14 to C36, C19 to C37, C27 to C38, C28 to C39, C44 to C40, C13 to C41, C20 to C42, C29 to C43, C30 to C44, C12 to C46, C21 to C47, C31 to C48, C32 to C49, C46 to C50, C10 to C51, C22 to C52, C33 to C53, C34 to C54, C47 to C55, C11 to C56, C8 to C57, C35 to C58, C36 to C59, C48 to C60, C3 to C61, C9 to C62, C37 to C63, C39 to C64, C23 to C65, C49 to C66, C38 to C67, C4 to C68, C40 to C69, C50 to C70, C2 to C71, C24 to C72, C41 to C73, C42 to C74, C51 to C75, C5 to C76, D8 to D10, D7 to D11, D2 to D12, D3 to D13, D4 to D14, D5 to D15, D6 to D16, D1 to D17, D10 to D8, IC19 to IC10, IC6 to IC11, IC7 to IC12, IC9 to IC13, IC10 to IC14, IC4 to IC16, IC8 to IC17, IC11 to IC18, IC12 to IC19, IC16 to IC20, IC5 to IC21, IC24 to IC22, IC13 to IC23, IC14 to IC24, IC17 to IC25, IC2 to IC26, IC18 to IC3, IC3 to IC4, IC23 to IC5, IC22 to IC6, IC21 to IC7, IC1 to IC8, IC20 to IC9, L2 to L1, L1 to L6, Q10 to Q1, Q1 to Q10, Q9 to Q2, Q8 to Q3, Q7 to Q4, Q2 to Q5, Q3 to Q6, Q4 to Q7, Q5 to Q8, Q6 to Q9, R35 to R1, R11 to R10, R18 to R11, R19 to R12, R20 to R13, R21 to R14, R30 to R15, R31 to R16, R12 to R17, R7 to R18, R14 to R19, R4 to R2, R15 to R20, R22 to R21, R23 to R22, R24 to R23, R25 to R24, R32 to R25, R33 to R26, R5 to R27, R8 to R28, R16 to R29, R37 to R3, R26 to R30, R27 to R31, R34 to R32, R9 to R33, R28 to R34, R10 to R35, R36 to R4, R6 to R5, R3 to R6, R38 to R7, R2 to R8, R13 to R9

Commit message: Adjusting footprints of components
Parts:
- C10, C11, C16, C17, C20, C21, C22, C23, C24, C26, C28, C32, C33, C34, C35, C36, C47, C48, C49, C50, C51, C62, C63, C64, C65, C66, C67, C68, C69, C70, C71: footprint C0603 -> PULSE_Library:C0603
- C13, C14, C15, C18, C19, C42, C43, C44, C45, C46, C57, C58, C59, C60, C61: footprint CAPC2012X145N -> PULSE_Library:CAPC2012X145N
- IC22, IC23, IC24, IC25, IC26, IC3, IC4: footprint SOIC127P600X175-8N -> PULSE_Library:SOIC127P600X175-8N
- IC8, IC9: footprint SOP50P490X110-10N -> PULSE_Library:SOP50P490X110-10N
- L1, L3, L4, L5, L6: footprint INDPM4440X200N -> PULSE_Library:INDPM4440X200N
- R1, R2, R3, R6, R7, R8: footprint RESC1608X55N -> PULSE_Library:RESC1608X55N
Changed lines of the file:
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@@
 			)
 		)
-		(property "Footprint" "RESC1608X55N"
+		(property "Footprint" "PULSE_Library:RESC1608X55N"
 			(at 80.01 441.63 0)
 			(effects
@@
 			)
 		)
-		(property "Footprint" "C0603"
+		(property "Footprint" "PULSE_Library:C0603"
 			(at 214.3 297.18 0)
 			(effects
@@
 			)
 		)
-		(property "Footprint" "C0603"
+		(property "Footprint" "PULSE_Library:C0603"
 			(at 503.86 97.79 0)
 			(effects
@@
 			)
 		)
-		(property "Footprint" "RESC1608X55N"
+		(property "Footprint" "PULSE_Library:RESC1608X55N"
 			(at 116.84 211.76 0)
 			(effects
@@
 			)
 		)
-		(property "Footprint" "C0603"
+		(property "Footprint" "PULSE_Library:C0603"
 			(at 500.05 220.98 0)
 			(effects
@@
 			)
 		)
-		(property "Footprint" "SOP50P490X110-10N"
+		(property "Footprint" "PULSE_Library:SOP50P490X110-10N"
 			(at 147.32 150.8 0)
 			(effects
@@
 			)
 		)
-		(property "Footprint" "C0603"
+		(property "Footprint" "PULSE_Library:C0603"
 			(at 599.11 110.49 0)
 			(effects
@@
 			)
 		)
-		(property "Footprint" "SOIC127P600X175-8N"
+		(property "Footprint" "PULSE_Library:SOIC127P600X175-8N"
 			(at 461.01 211.76 0)
 			(effects
@@
 			)
 		)
-		(property "Footprint" "INDPM4440X200N"
+		(property "Footprint" "PULSE_Library:INDPM4440X200N"
 			(at 414.35 231.14 0)
 			(effects
@@
 			)
 		)
-		(property "Footprint" "C0603"
+		(property "Footprint" "PULSE_Library:C0603"
 			(at 260.02 332.74 0)
 			(effects
@@
 			)
 		)
-		(property "Footprint" "RESC1608X55N"
+		(property "Footprint" "PULSE_Library:RESC1608X55N"
 			(at 125.73 211.76 0)
 			(effects
@@
 			)
 		)
-		(property "Footprint" "C0603"
+		(property "Footprint" "PULSE_Library:C0603"
 			(at 509.27 167.31 0)
 			(effects
@@
 			)
 		)
-		(property "Footprint" "C0603"
+		(property "Footprint" "PULSE_Library:C0603"
 			(at 252.4 106.68 0)
 			(effects
@@
 			)
 		)
-		(property "Footprint" "C0603"
+		(property "Footprint" "PULSE_Library:C0603"
 			(at 233.35 184.15 0)
 			(effects
@@
 			)
 		)
-		(property "Footprint" "C0603"
+		(property "Footprint" "PULSE_Library:C0603"
 			(at 71.12 454.33 0)
 			(effects
@@
 			)
 		)
-		(property "Footprint" "C0603"
+		(property "Footprint" "PULSE_Library:C0603"
 			(at 506.73 281.61 0)
 			(effects
@@
 			)
 		)
-		(property "Footprint" "CAPC2012X145N"
+		(property "Footprint" "PULSE_Library:CAPC2012X145N"
 			(at 383.54 219.38 0)
 			(effects
@@
 			)
 		)
-		(property "Footprint" "CAPC2012X145N"
+		(property "Footprint" "PULSE_Library:CAPC2012X145N"
 			(at 113.03 265.1 0)
 			(effects
@@
 			)
 		)
-		(property "Footprint" "CAPC2012X145N"
+		(property "Footprint" "PULSE_Library:CAPC2012X145N"
 			(at 454.66 220.65 0)
 			(effects
@@
 			)
 		)
-		(property "Footprint" "CAPC2012X145N"
+		(property "Footprint" "PULSE_Library:CAPC2012X145N"
 			(at 450.85 343.84 0)
 			(effects
@@
 			)
 		)
-		(property "Footprint" "C0603"
+		(property "Footprint" "PULSE_Library:C0603"
 			(at 498.78 279.4 0)
 			(effects
@@
 			)
 		)
-		(property "Footprint" "C0603"
+		(property "Footprint" "PULSE_Library:C0603"
 			(at 504.19 347.65 0)
 			(effects
@@
 			)
 		)
-		(property "Footprint" "CAPC2012X145N"
+		(property "Footprint" "PULSE_Library:CAPC2012X145N"
 			(at 110.49 347.65 0)
 			(effects
@@
 			)
 		)
-		(property "Footprint" "C0603"
+		(property "Footprint" "PULSE_Library:C0603"
 			(at 594.03 292.1 0)
 			(effects
@@
 			)
 		)
-		(property "Footprint" "C0603"
+		(property "Footprint" "PULSE_Library:C0603"
 			(at 295.91 351.46 0)
 			(effects
@@
 			)
 		)
-		(property "Footprint" "CAPC2012X145N"
+		(property "Footprint" "PULSE_Library:CAPC2012X145N"
 			(at 453.39 277.8 0)
 			(effects
@@
 			)
 		)
-		(property "Footprint" "INDPM4440X200N"
+		(property "Footprint" "PULSE_Library:INDPM4440X200N"
 			(at 419.43 50.8 0)
 			(effects
@@
 			)
 		)
-		(property "Footprint" "CAPC2012X145N"
+		(property "Footprint" "PULSE_Library:CAPC2012X145N"
 			(at 379.73 342.57 0)
 			(effects
@@
 			)
 		)
-		(property "Footprint" "CAPC2012X145N"
+		(property "Footprint" "PULSE_Library:CAPC2012X145N"
 			(at 140.97 407.34 0)
 			(effects
@@
 			)
 		)
-		(property "Footprint" "CAPC2012X145N"
+		(property "Footprint" "PULSE_Library:CAPC2012X145N"
 			(at 111.76 307.01 0)
 			(effects
@@
 			)
 		)
-		(property "Footprint" "CAPC2012X145N"
+		(property "Footprint" "PULSE_Library:CAPC2012X145N"
 			(at 384.81 162.23 0)
 			(effects
@@
 			)
 		)
-		(property "Footprint" "C0603"
+		(property "Footprint" "PULSE_Library:C0603"
 			(at 261.29 285.75 0)
 			(effects
@@
 			)
 		)
-		(property "Footprint" "SOIC127P600X175-8N"
+		(property "Footprint" "PULSE_Library:SOIC127P600X175-8N"
 			(at 99.06 445.44 0)
 			(effects
@@
 			)
 		)
-		(property "Footprint" "C0603"
+		(property "Footprint" "PULSE_Library:C0603"
 			(at 72.39 407.34 0)
 			(effects
@@
 			)
 		)
-		(property "Footprint" "C0603"
+		(property "Footprint" "PULSE_Library:C0603"
 			(at 252.4 62.23 0)
 			(effects
@@
 			)
 		)
-		(property "Footprint" "CAPC2012X145N"
+		(property "Footprint" "PULSE_Library:CAPC2012X145N"
 			(at 378.46 400.99 0)
 			(effects
@@
 			)
 		)
-		(property "Footprint" "CAPC2012X145N"
+		(property "Footprint" "PULSE_Library:CAPC2012X145N"
 			(at 382.27 276.53 0)
 			(effects
@@
 			)
 		)
-		(property "Footprint" "SOIC127P600X175-8N"
+		(property "Footprint" "PULSE_Library:SOIC127P600X175-8N"
 			(at 100.33 398.45 0)
 			(effects
@@
 			)
 		)
-		(property "Footprint" "INDPM4440X200N"
+		(property "Footprint" "PULSE_Library:INDPM4440X200N"
 			(at 418.16 107.95 0)
 			(effects
@@
 			)
 		)
-		(property "Footprint" "RESC1608X55N"
+		(property "Footprint" "PULSE_Library:RESC1608X55N"
 			(at 81.28 394.64 0)
 			(effects
@@
 			)
 		)
-		(property "Footprint" "RESC1608X55N"
+		(property "Footprint" "PULSE_Library:RESC1608X55N"
 			(at 133.35 167.31 0)
 			(effects
@@
 			)
 		)
-		(property "Footprint" "INDPM4440X200N"
+		(property "Footprint" "PULSE_Library:INDPM4440X200N"
 			(at 416.89 165.1 0)
 			(effects
@@
 			)
 		)
-		(property "Footprint" "C0603"
+		(property "Footprint" "PULSE_Library:C0603"
 			(at 505.13 40.64 0)
 			(effects
@@
 			)
 		)
-		(property "Footprint" "C0603"
+		(property "Footprint" "PULSE_Library:C0603"
 			(at 294.64 409.88 0)
 			(effects
@@
 			)
 		)
-		(property "Footprint" "C0603"
+		(property "Footprint" "PULSE_Library:C0603"
 			(at 600.38 53.34 0)
 			(effects
@@
 			)
 		)
-		(property "Footprint" "RESC1608X55N"
+		(property "Footprint" "PULSE_Library:RESC1608X55N"
 			(at 124.46 167.31 0)
 			(effects
@@
 			)
 		)
-		(property "Footprint" "C0603"
+		(property "Footprint" "PULSE_Library:C0603"
 			(at 597.84 167.64 0)
 			(effects
@@
 			)
 		)
-		(property "Footprint" "INDPM4440X200N"
+		(property "Footprint" "PULSE_Library:INDPM4440X200N"
 			(at 413.08 289.56 0)
 			(effects
@@
 			)
 		)
-		(property "Footprint" "C0603"
+		(property "Footprint" "PULSE_Library:C0603"
 			(at 595.3 233.68 0)
 			(effects
@@
 			)
 		)
-		(property "Footprint" "SOP50P490X110-10N"
+		(property "Footprint" "PULSE_Library:SOP50P490X110-10N"
 			(at 147.32 195.25 0)
 			(effects
@@
 			)
 		)
-		(property "Footprint" "SOIC127P600X175-8N"
+		(property "Footprint" "PULSE_Library:SOIC127P600X175-8N"
 			(at 487.68 334.95 0)
 			(effects
@@
 			)
 		)
-		(property "Footprint" "SOIC127P600X175-8N"
+		(property "Footprint" "PULSE_Library:SOIC127P600X175-8N"
 			(at 486.41 393.37 0)
 			(effects
@@
 			)
 		)
-		(property "Footprint" "C0603"
+		(property "Footprint" "PULSE_Library:C0603"
 			(at 300.99 171.12 0)
 			(effects
@@
 			)
 		)
-		(property "Footprint" "C0603"
+		(property "Footprint" "PULSE_Library:C0603"
 			(at 508 224.46 0)
 			(effects
@@
 			)
 		)
-		(property "Footprint" "C0603"
+		(property "Footprint" "PULSE_Library:C0603"
 			(at 298.45 285.42 0)
 			(effects
@@
 			)
 		)
-		(property "Footprint" "CAPC2012X145N"
+		(property "Footprint" "PULSE_Library:CAPC2012X145N"
 			(at 139.7 454.33 0)
 			(effects
@@
 			)
 		)
-		(property "Footprint" "CAPC2012X145N"
+		(property "Footprint" "PULSE_Library:CAPC2012X145N"
 			(at 449.58 402.26 0)
 			(effects
@@
 			)
 		)
-		(property "Footprint" "C0603"
+		(property "Footprint" "PULSE_Library:C0603"
 			(at 299.72 228.27 0)
 			(effects
@@
 			)
 		)
-		(property "Footprint" "C0603"
+		(property "Footprint" "PULSE_Library:C0603"
 			(at 502.92 406.07 0)
 			(effects
@@
 			)
 		)
-		(property "Footprint" "C0603"
+		(property "Footprint" "PULSE_Library:C0603"
 			(at 234.62 142.24 0)
 			(effects
@@
 			)
 		)
-		(property "Footprint" "C0603"
+		(property "Footprint" "PULSE_Library:C0603"
 			(at 502.59 154.94 0)
 			(effects
@@
 			)
 		)
-		(property "Footprint" "CAPC2012X145N"
+		(property "Footprint" "PULSE_Library:CAPC2012X145N"
 			(at 455.93 163.5 0)
 			(effects
@@
 			)
 		)
-		(property "Footprint" "SOIC127P600X175-8N"
+		(property "Footprint" "PULSE_Library:SOIC127P600X175-8N"
 			(at 462.28 154.61 0)
 			(effects
@@
 			)
 		)
-		(property "Footprint" "SOIC127P600X175-8N"
+		(property "Footprint" "PULSE_Library:SOIC127P600X175-8N"
 			(at 459.74 268.91 0)
 			(effects
@@
 			)
 		)
-		(property "Footprint" "C0603"
+		(property "Footprint" "PULSE_Library:C0603"
 			(at 213.03 344.17 0)
 			(effects
@@
 			)
 		)
-		(property "Footprint" "C0603"
+		(property "Footprint" "PULSE_Library:C0603"
 			(at 232.08 224.79 0)
 			(effects
