File: EPS_PDU.kicad_sch (KiCad schematic)
At the start: 0 parts

Commit message: PDU_SCHEMATICS_v01
Parts:
- added C1, C10, C16, C2, C21, C23, C31, C32, C38, C40, C46, C50, C53, C55, C57, C59, C6, C62, C65: 0.1μF, C0603, symbol Device:C_Small
- added C11, C17, C22, C24, C33, C34, C41, C42, C47, C5, C51, C56, C60, C63, C66: 47μF, GRT32ER60J107ME13L, symbol Device:C_Small
- added C12, C15, C20, C29, C3, C30, C35, C36, C45, C48, C54, C58, C61, C64, C8: 10μF, CAPC2012X145N, symbol Device:C_Small
- added C13, C19, C27, C28, C44: 4.7μF, C0805, symbol Device:C_Small
- added C14, C18, C25, C26, C43: 0.47μF, C0603, symbol Device:C_Small
- added C37, C39, C4, C49, C52, C7, C9: 1μF, C0603, symbol Device:C_Small
- added D1, D10, D2, D3, D4, D5, D6, D7, D8, D9: SMAJ16CA, Diode_SMD:D_SMA, symbol Diode:SMAJ16CA
- added IC1, IC20: INA226AIDGSR, SOP50P490X110-10N, symbol PDU_Library:INA226AIDGSR
- added IC10, IC15, IC4, IC7, IC9: MAX17523ATE+, QFN50P300X300X80-17N, symbol PDU_Library:MAX17523ATE+
- added IC11, IC12, IC16, IC19, IC21, IC22, IC23, IC5, IC6, IC8: LM74700QDBVRQ1, SOT95P280X145-6N, symbol PDU_Library:LM74700QDBVRQ1
- added IC13, IC24: L6982C50DR, SOIC127P600X175-8N, symbol PDU_Library:L6982C50DR
- added IC14, IC17, IC2: L6982C33DR, SOIC127P600X175-8N, symbol PDU_Library:L6982C33DR
- added IC18, IC3: MAX890LESA+, SOIC127P600X175-8N, symbol PDU_Library:MAX890LESA+
- added L1, L2, L3, L4, L5: 22μH, INDPM4440X200N, symbol Device:L_Small
- added Q1, Q10, Q2, Q3, Q4, Q5, Q6, Q7, Q8, Q9: DMN4035LQ-13, SOT96P240X110-3N, symbol PDU_Library:DMN4035LQ-13
- added R10, R28: 2mΩ, RESC3216X59N, symbol Device:R_Small_US
- added R11, R15, R19, R21, R23, R25, R31, R33, R7, R8: 305KΩ, Resistor_SMD:R_0603_1608Metric, symbol Device:R_Small_US
- added R12, R13, R14, R18, R20, R22, R24, R30, R32, R5: 2.2MΩ, RESC3216X59N, symbol Device:R_Small_US
- added R16, R26, R27, R34, R9: 6.12KΩ, Resistor_SMD:R_0603_1608Metric, symbol Device:R_Small_US
- added R2, R3, R37, R38: 10KΩ, RESC1608X55N, symbol Device:R_Small_US
- added R35, R4: 100KΩ, RESC1608X55N, symbol Device:R_Small_US
- added R36, R6: 1.38KΩ, Resistor_SMD:R_0603_1608Metric, symbol Device:R_Small_US
Connections:
- new net: IC18.8 (~{FAULT}), R35.1
- new net: C52.1, IC18.1 (IN_1), IC18.2 (IN_2), R35.2
- new net: C43.1, IC15.6 (IN_1), IC15.7 (IN_2), R30.1, R32.1
- new net: IC15.8 (OVLO), R30.2, R31.1
- new net: IC7.10 (SETI), R16.1
- new net: C19.2, C20.2, C21.2, D3.1 (A1), IC7.14 (OUT_1), IC7.15 (OUT_2), IC8.3 (EN), IC8.6 (ANODE), Q3.2 (S)
- new net: IC7.2 (CLHS), IC7.3 (CLTS1)
- new net: C18.1, IC7.6 (IN_1), IC7.7 (IN_2), R13.1, R14.1
- new net: IC7.8 (OVLO), R11.1, R13.2
- new net: IC7.9 (UVLO), R14.2, R15.1
- new net: C15.2, C16.2, C6.1, D2.1 (A1), IC3.6 (OUT_1), IC3.7 (OUT_2), IC6.3 (EN), IC6.6 (ANODE), Q2.2 (S)
- new net: C15.1, C6.2, D2.2 (A2), IC6.2 (GND)
- new net: C22.1, IC8.4 (CATHODE), Q3.3 (D)
- new net: IC8.5 (GATE), Q3.1 (G)
- new net: IC15.9 (UVLO), R32.2, R33.1
- new net: C46.1, IC16.1 (VCAP)
- new net: C44.2, C45.2, C46.2, D6.1 (A1), IC15.14 (OUT_1), IC15.15 (OUT_2), IC16.3 (EN), IC16.6 (ANODE), Q6.2 (S)
- new net: C57.1, IC20.2 (A0), IC20.6 (VS), R37.2, R38.2
- new net: C31.1, IC11.1 (VCAP)
- new net: C27.2, C29.2, C31.2, D4.1 (A1), IC11.3 (EN), IC11.6 (ANODE), IC9.14 (OUT_1), IC9.15 (OUT_2), Q4.2 (S)
- new net: C1.1, IC1.6 (VS), R2.2, R3.2
- new net: IC1.8 (VBUS), IC1.9 (IN-)
- new net: IC4.10 (SETI), R9.1
- new net: IC21.5 (GATE), Q8.1 (G)
- new net: C58.2, C59.2, D8.1 (A1), IC21.3 (EN), IC21.6 (ANODE), Q8.2 (S)
- new net: C60.1, IC21.4 (CATHODE), Q8.3 (D)
- new net: IC3.5 (SET), R6.1
- new net: C5.1, IC2.4 (VOUT/FB), L1.1, R10.2
- new net: C50.1, IC17.2 (BOOT)
- new net: C50.2, IC17.1 (SW), L5.2
- new net: IC5.5 (GATE), Q1.1 (G)
- new net: C10.2, C12.2, C13.2, D1.1 (A1), IC4.14 (OUT_1), IC4.15 (OUT_2), IC5.3 (EN), IC5.6 (ANODE), Q1.2 (S)
- new net: C11.1, IC5.4 (CATHODE), Q1.3 (D)
- new net: C49.1, IC17.3 (VCC)
- new net: C51.1, IC17.4 (VOUT/FB), L5.1
- new net: C48.1, IC17.5 (EN/CLKIN), IC17.7 (VIN)
- new net: C41.1, IC13.5 (EN/CLKIN), L3.1, R28.2
- new net: C38.2, IC13.8 (PGND), L3.2
- new net: IC19.5 (GATE), Q7.1 (G)
- new net: C53.1, C54.2, C55.2, D7.1 (A1), IC18.6 (OUT_1), IC18.7 (OUT_2), IC19.3 (EN), IC19.6 (ANODE), Q7.2 (S)
- new net: C56.1, IC19.4 (CATHODE), Q7.3 (D)
- new net: C55.1, IC19.1 (VCAP)
- new net: C4.1, IC2.3 (VCC)
- new net: C14.1, IC4.6 (IN_1), IC4.7 (IN_2), R12.1, R5.1
- new net: IC4.8 (OVLO), R12.2, R7.1
- new net: C62.1, IC22.1 (VCAP)
- new net: C61.2, C62.2, D9.1 (A1), IC22.3 (EN), IC22.6 (ANODE), Q9.2 (S)
- new net: C39.1, IC14.3 (VCC)
- new net: IC4.9 (UVLO), R5.2, R8.1
- new net: C42.1, IC14.4 (VOUT/FB), L4.1
- new net: C28.2, C30.2, C32.2, D5.1 (A1), IC10.14 (OUT_1), IC10.15 (OUT_2), IC12.3 (EN), IC12.6 (ANODE), Q5.2 (S)
- new net: IC23.5 (GATE), Q10.1 (G)
- new net: C64.2, C65.2, D10.1 (A1), IC23.3 (EN), IC23.6 (ANODE), Q10.2 (S)
- new net: C66.1, IC23.4 (CATHODE), Q10.3 (D)
- new net: IC10.8 (OVLO), R20.2, R21.1
- new net: C25.1, IC9.6 (IN_1), IC9.7 (IN_2), R18.1, R22.1
- new net: IC9.9 (UVLO), R22.2, R23.1
- new net: IC9.8 (OVLO), R18.2, R19.1
- new net: IC15.10 (SETI), R34.1
- new net: C63.1, IC22.4 (CATHODE), Q9.3 (D)
- new net: IC22.5 (GATE), Q9.1 (G)
- new net: C32.1, IC12.1 (VCAP)
- new net: C34.1, IC12.4 (CATHODE), Q5.3 (D)
- new net: IC12.5 (GATE), Q5.1 (G)
- new net: IC9.10 (SETI), R26.1
- new net: IC9.2 (CLHS), IC9.3 (CLTS1)
- new net: C53.2, C54.1, D7.2 (A2), IC19.2 (GND)
- new net: C35.1, IC13.2 (BOOT), IC13.4 (VOUT/FB)
- new net: IC11.5 (GATE), Q4.1 (G)
- new net: C33.1, IC11.4 (CATHODE), Q4.3 (D)
- new net: C21.1, IC8.1 (VCAP)
- new net: C37.1, IC13.6 (AGND)
- new net: IC10.10 (SETI), R27.1
- new net: C47.1, IC16.4 (CATHODE), Q6.3 (D)
- new net: C23.1, IC24.7 (VIN)
- new net: C23.2, IC24.8 (PGND), L2.2
- new net: C36.1, IC14.5 (EN/CLKIN), IC14.7 (VIN)
- new net: C2.2, IC2.1 (SW), L1.2
- new net: IC15.2 (CLHS), IC15.3 (CLTS1)
- new net: IC10.9 (UVLO), R24.2, R25.1
- new net: C16.1, IC6.1 (VCAP)
- new net: IC18.5 (SET), R36.1
- new net: C7.1, IC3.1 (IN_1), IC3.2 (IN_2), R4.2
- new net: C26.1, IC10.6 (IN_1), IC10.7 (IN_2), R20.1, R24.1
- new net: IC3.8 (~{FAULT}), R4.1
- new net: IC4.2 (CLHS), IC4.3 (CLTS1)
- new net: IC16.5 (GATE), Q6.1 (G)
- new net: C40.2, IC14.1 (SW), L4.2
- new net: C10.1, IC5.1 (VCAP)
- new net: C2.1, IC2.2 (BOOT)
- new net: C40.1, IC14.2 (BOOT)
- new net: IC10.2 (CLHS), IC10.3 (CLTS1)
- new net: C24.1, IC24.5 (EN/CLKIN), L2.1
- new net: C38.1, IC13.7 (VIN)
- new net: IC20.8 (VBUS), IC20.9 (IN-)
- new net: C8.1, IC24.2 (BOOT), IC24.4 (VOUT/FB)
- new net: C9.1, IC24.6 (AGND)
- new net: IC6.5 (GATE), Q2.1 (G)
- new net: C17.1, IC6.4 (CATHODE), Q2.3 (D)
- new net: C65.1, IC23.1 (VCAP)
- new net: C59.1, IC21.1 (VCAP)
- new net: C3.1, IC2.5 (EN/CLKIN), IC2.7 (VIN)
- new net EN: IC10.13 (EN), IC15.13 (EN), IC4.13 (EN), IC7.13 (EN), IC9.13 (EN)
- new net FLAG: IC10.12 (~{FLAG}), IC15.12 (~{FLAG}), IC4.12 (~{FLAG}), IC7.12 (~{FLAG}), IC9.12 (~{FLAG})
- new net GND: C1.2, C11.2, C12.1, C13.1, C14.2, C17.2, C18.2, C19.1, C20.1, C22.2, C24.2, C25.2, C26.2, C27.1, C28.1, C29.1, C3.2, C30.1, C33.2, C34.2, C35.2, C36.2, C37.2, C39.2, C4.2, C41.2, C42.2, C43.2, C44.1, C45.1, C47.2, C48.2, C49.2, C5.2, C51.2, C52.2, C56.2, C57.2, C58.1, C60.2, C61.1, C63.2, C64.1, C66.2, C7.2, C8.2, C9.2, D1.2 (A2), D10.2 (A2), D3.2 (A2), D4.2 (A2), D5.2 (A2), D6.2 (A2), D8.2 (A2), D9.2 (A2), IC1.1 (A1), IC1.2 (A0), IC1.7 (GND), IC10.1 (CLTS_MODE), IC10.11 (GND), IC10.17 (EP), IC10.4 (CLTS2), IC11.2 (GND), IC12.2 (GND), IC13.1 (SW), IC13.3 (VCC), IC14.6 (AGND), IC14.8 (PGND), IC15.1 (CLTS_MODE), IC15.11 (GND), IC15.17 (EP), IC15.4 (CLTS2), IC16.2 (GND), IC17.6 (AGND), IC17.8 (PGND), IC18.4 (GND), IC2.6 (AGND), IC2.8 (PGND), IC20.1 (A1), IC20.7 (GND), IC21.2 (GND), IC22.2 (GND), IC23.2 (GND), IC24.1 (SW), IC24.3 (VCC), IC3.4 (GND), IC4.1 (CLTS_MODE), IC4.11 (GND), IC4.17 (EP), IC4.4 (CLTS2), IC5.2 (GND), IC7.1 (CLTS_MODE), IC7.11 (GND), IC7.17 (EP), IC7.4 (CLTS2), IC8.2 (GND), IC9.1 (CLTS_MODE), IC9.11 (GND), IC9.17 (EP), IC9.4 (CLTS2), R11.2, R15.2, R16.2, R19.2, R21.2, R23.2, R25.2, R26.2, R27.2, R31.2, R33.2, R34.2, R36.2, R6.2, R7.2, R8.2, R9.2
- new net HVEN_: IC10.5 (~{HVEN}), IC15.5 (~{HVEN}), IC4.5 (~{HVEN}), IC7.5 (~{HVEN}), IC9.5 (~{HVEN})
- new net ON_: IC18.3 (~{ON}), IC3.3 (~{ON})
- new net RIEN_: IC10.16 (~{RIEN}), IC15.16 (~{RIEN}), IC4.16 (~{RIEN}), IC7.16 (~{RIEN}), IC9.16 (~{RIEN})
- new net SCL2: IC1.5 (SCL), IC20.5 (SCL), R2.1, R38.1
- new net SDA2: IC1.4 (SDA), IC20.4 (SDA), R3.1, R37.1
- no-connect marks 0 -> 2
Other:
- company: EPFL Spacecraft Team -> (none)

Commit message: modifications on PDU
Parts:
- removed C10, C21, C31, C32, C46: 0.1μF, C0603, symbol Device:C_Small
- removed C11, C22, C33, C34, C47: 47μF, GRT32ER60J107ME13L, symbol Device:C_Small
- removed C12, C20, C30, C45: 10μF, CAPC2012X145N, symbol Device:C_Small
- removed C13, C44: 4.7μF, C0805, symbol Device:C_Small
- removed D1, D3, D4, D5, D6: SMAJ16CA, Diode_SMD:D_SMA, symbol Diode:SMAJ16CA
- removed IC11, IC12, IC16, IC5, IC8: LM74700QDBVRQ1, SOT95P280X145-6N, symbol PDU_Library:LM74700QDBVRQ1
- removed Q1, Q3, Q4, Q5, Q6: DMN4035LQ-13, SOT96P240X110-3N, symbol PDU_Library:DMN4035LQ-13
- C29: value 10μF -> 4.7μF; footprint CAPC2012X145N -> C0805; Height 1.45 -> 1.1; Manufacturer_Name YAGEO -> KEMET; Manufacturer_Part_Number CC0805KKX7R7BB106 -> C0805C475K4RACAUTO; Mouser Part Number 603-CC0805KKX77BB106 -> 80-C0805C475K4RAUTO; Mouser Price/Stock https://www.mouser.co.uk/ProductDetail/YAGEO/CC0805KKX7R7BB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 -> https://www.mouser.co.uk/ProductDetail/KEMET/C0805C475K4RAC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
- renumbered C6 to C?, C50 to C?, C55 to C?, C4 to C?, C57 to C?, C62 to C?, C52 to C?, C5 to C?, C39 to C?, C42 to C?, C58 to C?, C19 to C?, C27 to C?, C48 to C?, C35 to C?, C37 to C?, C64 to C?, C23 to C?, C25 to C?, C36 to C?, C63 to C?, C41 to C?, C15 to C?, C61 to C?, C16 to C?, C7 to C?, C1 to C?, C56 to C?, C66 to C?, C60 to C?, C18 to C?, C2 to C?, C40 to C?, C38 to C?, C51 to C?, C14 to C?, C49 to C?, C26 to C?, C54 to C?, C8 to C?, C43 to C?, C9 to C?, C24 to C?, C59 to C?, C3 to C?, C17 to C?, C53 to C?, C65 to C?, D10 to D?, D2 to D?, D8 to D?, D7 to D?, D9 to D?, IC7 to IC?, IC1 to IC?, IC17 to IC?, IC22 to IC?, IC9 to IC?, IC19 to IC?, IC15 to IC?, IC18 to IC?, IC3 to IC?, IC4 to IC?, IC10 to IC?, IC20 to IC?, IC13 to IC?, IC24 to IC?, IC6 to IC?, IC23 to IC?, IC21 to IC?, IC2 to IC?, IC14 to IC?, L3 to L?, L1 to L?, L5 to L?, L4 to L?, L2 to L?, Q8 to Q?, Q7 to Q?, Q10 to Q?, Q9 to Q?, Q2 to Q?, R35 to R?, R30 to R?, R32 to R?, R37 to R?, R9 to R?, R6 to R?, R10 to R?, R31 to R?, R38 to R?, R12 to R?, R5 to R?, R7 to R?, R21 to R?, R22 to R?, R19 to R?, R15 to R?, R34 to R?, R28 to R?, R23 to R?, R33 to R?, R13 to R?, R27 to R?, R11 to R?, R14 to R?, R25 to R?, R20 to R?, R26 to R?, R16 to R?, R4 to R?, R2 to R?, R3 to R?, R24 to R?, R18 to R?, R8 to R?, R36 to R?
Connections:
- net RIEN_ is gone; now on net GND: IC?.16 (~{RIEN}), IC?.16 (~{RIEN}), IC?.16 (~{RIEN}), IC?.16 (~{RIEN}), IC?.16 (~{RIEN})
- net GND: now also C28.2, C29.2, C?.2, C?.2; no longer C28.1, C29.1, C?.1, C?.1
- net at IC?.14 (OUT_1), IC?.15 (OUT_2): now also C?.1, C?.1, IC?.2 (BOOT), IC?.4 (VOUT/FB); no longer C?.2
- net at IC?.14 (OUT_1), IC?.15 (OUT_2): now also C28.1, C?.1, IC?.5 (EN/CLKIN), IC?.7 (VIN)
- net at IC?.14 (OUT_1), IC?.15 (OUT_2): now also C?.1, C?.1, IC?.2 (BOOT), IC?.4 (VOUT/FB); no longer C29.2, C?.2
- net at IC?.14 (OUT_1), IC?.15 (OUT_2): now also C?.1, C?.1, IC?.5 (EN/CLKIN), IC?.7 (VIN)
- net at IC?.14 (OUT_1), IC?.15 (OUT_2): now also C29.1, C?.1, IC?.5 (EN/CLKIN), IC?.7 (VIN); no longer C28.2
- removed net EN: IC?.13 (EN), IC?.13 (EN), IC?.13 (EN), IC?.13 (EN), IC?.13 (EN)
- new net EN_3.3V_1: IC?.13 (EN)
- new net EN_3.3V_2: IC?.13 (EN)
- new net EN_3.3V_3: IC?.13 (EN)
- new net EN_5V_1: IC?.13 (EN)
- new net EN_5V_2: IC?.13 (EN)
Other:
- moved on the sheet: C27, C?, IC?, L?, R?

Commit message: Final schematics pdu
Parts:
- removed C? (x9): 0.1μF, C0603, symbol Device:C_Small
- removed C? (x7): 1μF, C0603, symbol Device:C_Small
- removed C? (x7): 47μF, GRT32ER60J107ME13L, symbol Device:C_Small
- removed C?: 4.7μF, C0805, symbol Device:C_Small
- removed C? (x7): 10μF, CAPC2012X145N, symbol Device:C_Small
- removed C? (x5): 0.47μF, C0603, symbol Device:C_Small
- removed D? (x2): SMAJ16CA, Diode_SMD:D_SMA, symbol Diode:SMAJ16CA
- removed IC? (x4): MAX17523ATE+, QFN50P300X300X80-17N, symbol PDU_Library:MAX17523ATE+
- removed IC? (x2): L6982C33DR, SOIC127P600X175-8N, symbol PDU_Library:L6982C33DR
- removed IC? (x2): LM74700QDBVRQ1, SOT95P280X145-6N, symbol PDU_Library:LM74700QDBVRQ1
- removed IC? (x2): MAX890LESA+, SOIC127P600X175-8N, symbol PDU_Library:MAX890LESA+
- removed IC?: L6982C50DR, SOIC127P600X175-8N, symbol PDU_Library:L6982C50DR
- removed L? (x4): 22μH, INDPM4440X200N, symbol Device:L_Small
- removed Q? (x2): DMN4035LQ-13, SOT96P240X110-3N, symbol PDU_Library:DMN4035LQ-13
- removed R? (x2): 100KΩ, RESC1608X55N, symbol Device:R_Small_US
- removed R? (x10): 2.2MΩ, RESC3216X59N, symbol Device:R_Small_US
- removed R? (x5): 6.12KΩ, Resistor_SMD:R_0603_1608Metric, symbol Device:R_Small_US
- removed R? (x2): 1.38KΩ, Resistor_SMD:R_0603_1608Metric, symbol Device:R_Small_US
- removed R?: 2mΩ, RESC3216X59N, symbol Device:R_Small_US
- removed R? (x10): 305KΩ, Resistor_SMD:R_0603_1608Metric, symbol Device:R_Small_US
- added C10, C17, C22, C32, C42: 10μF, CAPC2012X145N, symbol Device:C_Small
- added C11, C18, C23, C33, C36, C37, C38, C41: 1μF, C0603, symbol Device:C_Small
- added C13, C19, C24, C34, C40: 0.1μF, C0603, symbol Device:C_Small
- added C14, C16, C21, C26, C43: 0.47μF, C0603, symbol Device:C_Small
- added C15, C20, C25, C35, C39: 47μF, GRT32ER60J107ME13L, symbol Device:C_Small
- added C30, C31: 4.7μF, C0805, symbol Device:C_Small
- added D10, D11, D12, D8, D9: SMAJ16CA, Diode_SMD:D_SMA, symbol Diode:SMAJ16CA
- added IC10, IC11, IC9: TPS25940ARVCR, PULSE_Library:QFN50P300X400X80-21N, symbol PULSE_Library:TPS25940ARVCR
- added IC12, IC5, IC7, IC8: MAX17523ATE+, QFN50P300X300X80-17N, symbol PDU_Library:MAX17523ATE+
- added IC25: L6982C50DR, SOIC127P600X175-8N, symbol PDU_Library:L6982C50DR
- added IC3, IC6: L6982C33DR, SOIC127P600X175-8N, symbol PDU_Library:L6982C33DR
- added L3, L4, L5, L6: 22μH, INDPM4440X200N, symbol Device:L_Small
- added R10, R16, R21, R7, R8: 305KΩ, Resistor_SMD:R_0603_1608Metric, symbol Device:R_Small_US
- added R11: 2mΩ, RESC3216X59N, symbol Device:R_Small_US
- added R12, R13, R15, R17, R20, R22, R45, R46, R5, R6: 2.2MΩ, RESC3216X59N, symbol Device:R_Small_US
- added R14, R19, R24, R44, R9: 6.12KΩ, Resistor_SMD:R_0603_1608Metric, symbol Device:R_Small_US
- added R18, R23, R25, R26, R27: 583KΩ, Resistor_SMD:R_0805_2012Metric_Pad1.20x1.40mm_HandSolder, symbol Device:R_Small_US
- added R28, R35, R43: 22.3KΩ, Resistor_SMD:R_0805_2012Metric_Pad1.20x1.40mm_HandSolder, symbol Device:R_Small_US
- added R29, R34, R42: 31.2KΩ, Resistor_SMD:R_0603_1608Metric, symbol Device:R_Small_US
- added R30, R32, R40: 264KΩ, Resistor_SMD:R_0805_2012Metric_Pad1.20x1.40mm_HandSolder, symbol Device:R_Small_US
- added R31, R33, R41: 20.8KΩ, Resistor_SMD:R_0805_2012Metric_Pad1.20x1.40mm_HandSolder, symbol Device:R_Small_US
- gave numbers to parts that had none: 4
Connections:
- net HVEN_ is gone; now on net GND: IC4.5 (~{HVEN})
- net EN_3.3V_1: now also IC12.13 (EN); no longer IC4.13 (EN)
- net EN_3.3V_2: now also IC4.13 (EN)
- net EN_3.3V_3: now also IC5.13 (EN)
- net EN_5V_1: now also IC7.13 (EN)
- net EN_5V_2: now also C35.1, IC25.5 (EN/CLKIN), IC8.13 (EN), L5.1
- net GND: now also C10.2, C11.2, C14.2, C15.2, C16.2, C17.2, C18.2, C20.2, C21.2, C22.2, C23.2, C25.2, C26.2, C30.2, C31.2, C32.2, C33.2, C35.2, C39.2, C41.2, C42.2, C43.2, D10.1 (A1), D11.1 (A1), D12.1 (A1), D8.1 (A1), D9.1 (A1), IC10.16 (GND), IC11.16 (GND), IC12.1 (CLTS_MODE), IC12.11 (GND), IC12.16 (~{RIEN}), IC12.17 (EP), IC12.4 (CLTS2), IC12.5 (~{HVEN}), IC25.1 (SW), IC25.3 (VCC), IC3.6 (AGND), IC3.8 (PGND), IC5.1 (CLTS_MODE), IC5.11 (GND), IC5.16 (~{RIEN}), IC5.17 (EP), IC5.4 (CLTS2), IC5.5 (~{HVEN}), IC6.6 (AGND), IC6.8 (PGND), IC7.1 (CLTS_MODE), IC7.11 (GND), IC7.16 (~{RIEN}), IC7.17 (EP), IC7.4 (CLTS2), IC7.5 (~{HVEN}), IC8.1 (CLTS_MODE), IC8.11 (GND), IC8.16 (~{RIEN}), IC8.17 (EP), IC8.4 (CLTS2), IC8.5 (~{HVEN}), IC9.16 (GND), R10.2, R14.2, R16.2, R18.2, R19.2, R21.2, R23.2, R24.2, R25.2, R26.2, R27.2, R28.1, R29.2, R34.2, R35.1, R42.2, R43.1, R44.2, R7.2, R8.2, R9.2
- net at IC24.2 (BOOT), IC24.4 (VOUT/FB): now also C22.1, C30.1, IC7.14 (OUT_1), IC7.15 (OUT_2)
- net +3.3V: now reaches C?.1, IC?.2 (A0), IC?.6 (VS), R?.2, R?.2
- net +3.3V: now also C?.1, IC?.6 (VS), R?.2, R?.2
- net 3.3V_1+: now reaches IC?.10 (IN+)
- net 3.3V_1+: now also IC?.4 (VOUT/FB), IC?.8 (VBUS), C39.1, L6.1, R11.2
- net 3.3V_1: now reaches IC?.9 (IN-)
- net 3.3V_1: now also R11.1; no longer IC?.8 (VBUS)
- net at IC4.10 (SETI): now also R9.1
- net V_bat_in: now reaches C?.2, C?.2, D?.1 (A1), IC?.3 (EN), IC?.6 (ANODE), Q?.2 (S)
- net V_bat_in: now also C?.2, C?.2, C?.2, C?.2, D?.1 (A1), D?.1 (A1), IC4.6 (IN_1), IC4.7 (IN_2), IC?.3 (EN), IC?.3 (EN), IC?.6 (ANODE), IC?.6 (ANODE), Q?.2 (S), Q?.2 (S), C14.1, C16.1, C21.1, C26.1, C43.1, D10.2 (A2), D11.2 (A2), D12.2 (A2), D8.2 (A2), D9.2 (A2), IC10.10 (IN_2), IC10.11 (IN_3), IC10.12 (IN_4), IC10.13 (IN_5), IC10.9 (IN_1), IC11.10 (IN_2), IC11.11 (IN_3), IC11.12 (IN_4), IC11.13 (IN_5), IC11.9 (IN_1), IC12.6 (IN_1), IC12.7 (IN_2), IC5.6 (IN_1), IC5.7 (IN_2), IC7.6 (IN_1), IC7.7 (IN_2), IC8.6 (IN_1), IC8.7 (IN_2), IC9.10 (IN_2), IC9.11 (IN_3), IC9.12 (IN_4), IC9.13 (IN_5), IC9.9 (IN_1), R12.1, R13.1, R15.1, R17.1, R20.1, R22.1, R30.1, R32.1, R40.1, R45.1, R46.1, R5.1, R6.1
- net V_bat_out1: now reaches C?.1, IC?.4 (CATHODE), Q?.3 (D)
- net 3.3V_2: now reaches L1.1
- net 3.3V_2: now also C15.1, IC3.4 (VOUT/FB); no longer IC?.4 (VOUT/FB)
- net at C28.1: now also IC4.14 (OUT_1), IC4.15 (OUT_2), C10.1, IC3.5 (EN/CLKIN), IC3.7 (VIN)
- net 5V_1+: now reaches R?.2
- net 5V_1+: now also IC24.5 (EN/CLKIN), IC?.10 (IN+), IC?.8 (VBUS), C25.1, L4.1
- net at IC?.3 (VCC): now also C41.1
- net at IC4.8 (OVLO): now also R12.2, R7.1
- net at IC4.9 (UVLO): now also R26.1, R5.2
- net V_bat_out3: now reaches C?.1, IC?.4 (CATHODE), Q?.3 (D)
- net 5V_1: now reaches R?.1
- net 5V_1: now also IC?.9 (IN-)
- net V_bat_out2: now reaches C?.1, IC?.4 (CATHODE), Q?.3 (D)
- net at C27.1: now also IC?.5 (EN/CLKIN), IC?.7 (VIN), C42.1, IC12.14 (OUT_1), IC12.15 (OUT_2)
- net at C29.1: now also C17.1, IC5.14 (OUT_1), IC5.15 (OUT_2), IC6.5 (EN/CLKIN), IC6.7 (VIN)
- net at IC24.7 (VIN): now also C24.1
- net at IC24.8 (PGND): now also C24.2, L4.2
- net at L1.2: now also C13.2, IC3.1 (SW); no longer IC?.1 (SW)
- net at IC?.2 (BOOT): now also C40.1
- net at IC24.6 (AGND): now also C23.1
- net FLAG: no longer names the net of IC4.12 (~{FLAG})
- new net: R30.2, R31.1
- new net: IC12.10 (SETI), R44.1
- new net: C19.2, IC6.1 (SW), L3.2
- new net: IC7.8 (OVLO), R15.2, R16.1
- new net: IC5.8 (OVLO), R10.1, R13.2
- new net: C36.2, IC9.1 (DEVSLP), IC9.17 (ILIM), R28.2
- new net: IC9.15 (OVP), R29.1, R31.2
- new net: IC7.9 (UVLO), R17.2, R23.1
- new net: IC8.10 (SETI), R24.1
- new net: C31.1, C32.1, IC25.2 (BOOT), IC25.4 (VOUT/FB), IC8.14 (OUT_1), IC8.15 (OUT_2)
- new net: IC8.2 (CLHS), IC8.3 (CLTS1)
- new net: IC8.8 (OVLO), R20.2, R21.1
- new net: IC8.9 (UVLO), R18.1, R22.2
- new net: C33.1, IC25.6 (AGND)
- new net: C34.1, IC25.7 (VIN)
- new net: C34.2, IC25.8 (PGND), L5.2
- new net: C19.1, IC6.2 (BOOT)
- new net: IC12.9 (UVLO), R27.1, R46.2
- new net: R32.2, R33.1
- new net: IC10.15 (OVP), R33.2, R34.1
- new net: C38.2, IC11.1 (DEVSLP), IC11.17 (ILIM), R43.2
- new net: C18.1, IC6.3 (VCC)
- new net: IC11.15 (OVP), R41.2, R42.1
- new net: C37.2, IC10.1 (DEVSLP), IC10.17 (ILIM), R35.2
- new net: C11.1, IC3.3 (VCC)
- new net: C13.1, IC3.2 (BOOT)
- new net: C40.2, IC?.1 (SW), L6.2
- new net: IC12.2 (CLHS), IC12.3 (CLTS1)
- new net: IC12.8 (OVLO), R45.2, R8.1
- new net: IC5.10 (SETI), R14.1
- new net: IC7.10 (SETI), R19.1
- new net: IC7.2 (CLHS), IC7.3 (CLTS1)
- new net: IC5.2 (CLHS), IC5.3 (CLTS1)
- new net: IC5.9 (UVLO), R25.1, R6.2
- new net: R40.2, R41.1
- new net 3.3V_3: C20.1, IC6.4 (VOUT/FB), L3.1
- new net EN_DEPLOY: IC10.14 (EN), IC11.14 (EN), IC9.14 (EN)
- new net SP BackUP Deploymnet Bus: C36.1, IC9.4 (OUT_1), IC9.5 (OUT_2), IC9.6 (OUT_3), IC9.7 (OUT_4), IC9.8 (OUT_5)
- new net SP Deploymnet Bus: C38.1, IC11.4 (OUT_1), IC11.5 (OUT_2), IC11.6 (OUT_3), IC11.7 (OUT_4), IC11.8 (OUT_5)
- new net UHF_Antenna_deploy: C37.1, IC10.4 (OUT_1), IC10.5 (OUT_2), IC10.6 (OUT_3), IC10.7 (OUT_4), IC10.8 (OUT_5)
- no-connect marks 2 -> 25
Other:
- note added: "OV : 10 V UV : 6 V ILIM : 1 A"
- note added: "OV : 10 V UV : 6 V ILIM : 4 A"
- moved on the sheet: C27, C?, D?, IC24, IC4, IC?, L1, Q?, R?

Commit message: lastest
Parts:
- removed C13, C24: 0.1μF, C0603, symbol Device:C_Small
- removed C14, C21: 0.47μF, C0603, symbol Device:C_Small
- removed C15, C20, C25: 47μF, GRT32ER60J107ME13L, symbol Device:C_Small
- removed C22: 10μF, CAPC2012X145N, symbol Device:C_Small
- removed C23, C38: 1μF, C0603, symbol Device:C_Small
- removed C29: 4.7μF, C0805, symbol Device:C_Small
- removed D10, D8, D9: SMAJ16CA, Diode_SMD:D_SMA, symbol Diode:SMAJ16CA
- removed IC10, IC11, IC9: TPS25940ARVCR, PULSE_Library:QFN50P300X400X80-21N, symbol PULSE_Library:TPS25940ARVCR
- removed IC25: L6982C50DR, SOIC127P600X175-8N, symbol PDU_Library:L6982C50DR
- removed IC3, IC6: L6982C33DR, SOIC127P600X175-8N, symbol PDU_Library:L6982C33DR
- removed IC5, IC7, IC8: MAX17523ATE+, QFN50P300X300X80-17N, symbol PDU_Library:MAX17523ATE+
- removed L6: 22μH, INDPM4440X200N, symbol Device:L_Small
- removed R34, R42: 31.2KΩ, Resistor_SMD:R_0603_1608Metric, symbol Device:R_Small_US
- removed R40: 264KΩ, Resistor_SMD:R_0805_2012Metric_Pad1.20x1.40mm_HandSolder, symbol Device:R_Small_US
- removed R41: 20.8KΩ, Resistor_SMD:R_0805_2012Metric_Pad1.20x1.40mm_HandSolder, symbol Device:R_Small_US
- removed R43: 22.3KΩ, Resistor_SMD:R_0805_2012Metric_Pad1.20x1.40mm_HandSolder, symbol Device:R_Small_US
- removed R44: 6.12KΩ, Resistor_SMD:R_0603_1608Metric, symbol Device:R_Small_US
- removed R45, R46, R6: 2.2MΩ, RESC3216X59N, symbol Device:R_Small_US
- removed R7, R8: 305KΩ, Resistor_SMD:R_0603_1608Metric, symbol Device:R_Small_US
- added C44, C45, C46, C57, C58, C59, C60, C61: 10μF, PULSE_Library:CAPC2012X145N, symbol Device:C_Small
- added C47, C48, C49, C50, C51, C65, C67, C69, C70, C71: 0.1μF, PULSE_Library:C0603, symbol Device:C_Small
- added C52, C53, C54, C55, C56, C72, C73, C74, C75, C76: 47μF, GRT32ER60J107ME13L, symbol Device:C_Small
- added C62, C63, C64, C66, C68: 1μF, PULSE_Library:C0603, symbol Device:C_Small
- added D13, D14, D15, D16, D17: SMAJ16CA, Diode_SMD:D_SMA, symbol Diode:SMAJ16CA
- added IC10, IC11, IC17, IC18, IC19, IC20, IC21: LM74700QDBVRQ1, SOT95P280X145-6N, symbol PDU_Library:LM74700QDBVRQ1
- added IC13, IC14, IC15: MAX17523ATE+, QFN50P300X300X80-17N, symbol PDU_Library:MAX17523ATE+
- added IC23: L6982C50DR, PULSE_Library:SOIC127P600X175-8N, symbol PDU_Library:L6982C50DR
- added IC24, IC25: L6982C33DR, PULSE_Library:SOIC127P600X175-8N, symbol PDU_Library:L6982C33DR
- added IC3, IC4: MAX890LESA+, PULSE_Library:SOIC127P600X175-8N, symbol PDU_Library:MAX890LESA+
- added L1: 22μH, PULSE_Library:INDPM4440X200N, symbol Device:L_Small
- added Q10, Q4, Q5, Q6, Q7, Q8, Q9: DMN4035LQ-13, SOT96P240X110-3N, symbol PDU_Library:DMN4035LQ-13
- added R1, R2: 100KΩ, PULSE_Library:RESC1608X55N, symbol Device:R_Small_US
- added R4: 1.38KΩ, Resistor_SMD:R_0603_1608Metric, symbol Device:R_Small_US
- C10: value 10μF -> 1μF; footprint CAPC2012X145N -> PULSE_Library:C0603; Height 1.45 -> 0.87; Manufacturer_Name YAGEO -> KEMET; Manufacturer_Part_Number CC0805KKX7R7BB106 -> C0603X105K4RACAUTO; Mouser Part Number 603-CC0805KKX77BB106 -> 80-C0603X105K4RAUTO; Mouser Price/Stock https://www.mouser.co.uk/ProductDetail/YAGEO/CC0805KKX7R7BB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 -> https://www.mouser.com/Search/Refine.aspx?Keyword=80-C0603X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
- C11: footprint C0603 -> PULSE_Library:C0603
- C13, C14, C15: renamed from C?; footprint CAPC2012X145N -> PULSE_Library:CAPC2012X145N
- C16, C26: value 0.47μF -> 0.1μF; footprint C0603 -> PULSE_Library:C0603; Manufacturer_Part_Number C0603X474J4RACAUTO -> C0603C104K4NACAUTO; Mouser Part Number 80-C0603X474J4RAUTO -> 80-C0603C104K4NAUTO; Mouser Price/Stock https://www.mouser.co.uk/ProductDetail/KEMET/C0603X474J4RAC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 -> https://www.mouser.co.uk/ProductDetail/KEMET/C0603C104K4NAC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
- C17: value 10μF -> 0.1μF; footprint CAPC2012X145N -> PULSE_Library:C0603; Height 1.45 -> 0.87; Manufacturer_Name YAGEO -> KEMET; Manufacturer_Part_Number CC0805KKX7R7BB106 -> C0603C104K4NACAUTO; Mouser Part Number 603-CC0805KKX77BB106 -> 80-C0603C104K4NAUTO; Mouser Price/Stock https://www.mouser.co.uk/ProductDetail/YAGEO/CC0805KKX7R7BB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 -> https://www.mouser.co.uk/ProductDetail/KEMET/C0603C104K4NAC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
- C18: value 1μF -> 10μF; footprint C0603 -> PULSE_Library:CAPC2012X145N; Height 0.87 -> 1.45; Manufacturer_Name KEMET -> YAGEO; Manufacturer_Part_Number C0603X105K4RACAUTO -> CC0805KKX7R7BB106; Mouser Part Number 80-C0603X105K4RAUTO -> 603-CC0805KKX77BB106; Mouser Price/Stock https://www.mouser.com/Search/Refine.aspx?Keyword=80-C0603X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 -> https://www.mouser.co.uk/ProductDetail/YAGEO/CC0805KKX7R7BB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
- C19: value 0.1μF -> 10μF; footprint C0603 -> PULSE_Library:CAPC2012X145N; Height 0.87 -> 1.45; Manufacturer_Name KEMET -> YAGEO; Manufacturer_Part_Number C0603C104K4NACAUTO -> CC0805KKX7R7BB106; Mouser Part Number 80-C0603C104K4NAUTO -> 603-CC0805KKX77BB106; Mouser Price/Stock https://www.mouser.co.uk/ProductDetail/KEMET/C0603C104K4NAC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 -> https://www.mouser.co.uk/ProductDetail/YAGEO/CC0805KKX7R7BB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
- C20, C21, C22, C23, C24: renamed from C?; footprint C0603 -> PULSE_Library:C0603
- C28: value 4.7μF -> 0.1μF; footprint C0805 -> PULSE_Library:C0603; Height 1.1 -> 0.87; Manufacturer_Part_Number C0805C475K4RACAUTO -> C0603C104K4NACAUTO; Mouser Part Number 80-C0805C475K4RAUTO -> 80-C0603C104K4NAUTO; Mouser Price/Stock https://www.mouser.co.uk/ProductDetail/KEMET/C0805C475K4RAC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 -> https://www.mouser.co.uk/ProductDetail/KEMET/C0603C104K4NAC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
- C30, C31: value 4.7μF -> 47μF; footprint C0805 -> GRT32ER60J107ME13L; Height 1.1 -> 2.7; Manufacturer_Name KEMET -> Murata Electronics; Manufacturer_Part_Number C0805C475K4RACAUTO -> GRT32EC81C476KE13L; Mouser Part Number 80-C0805C475K4RAUTO -> 81-GRT32EC81C476KE3L; Mouser Price/Stock https://www.mouser.co.uk/ProductDetail/KEMET/C0805C475K4RAC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 -> https://www.mouser.co.uk/ProductDetail/Murata-Electronics/G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
- C32: value 10μF -> 0.47μF; footprint CAPC2012X145N -> PULSE_Library:C0603; Height 1.45 -> 0.87; Manufacturer_Name YAGEO -> KEMET; Manufacturer_Part_Number CC0805KKX7R7BB106 -> C0603X474J4RACAUTO; Mouser Part Number 603-CC0805KKX77BB106 -> 80-C0603X474J4RAUTO; Mouser Price/Stock https://www.mouser.co.uk/ProductDetail/YAGEO/CC0805KKX7R7BB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 -> https://www.mouser.co.uk/ProductDetail/KEMET/C0603X474J4RAC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
- C33, C36: value 1μF -> 0.47μF; footprint C0603 -> PULSE_Library:C0603; Manufacturer_Part_Number C0603X105K4RACAUTO -> C0603X474J4RACAUTO; Mouser Part Number 80-C0603X105K4RAUTO -> 80-C0603X474J4RAUTO; Mouser Price/Stock https://www.mouser.com/Search/Refine.aspx?Keyword=80-C0603X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 -> https://www.mouser.co.uk/ProductDetail/KEMET/C0603X474J4RAC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
- C34: value 0.1μF -> 0.47μF; footprint C0603 -> PULSE_Library:C0603; Manufacturer_Part_Number C0603C104K4NACAUTO -> C0603X474J4RACAUTO; Mouser Part Number 80-C0603C104K4NAUTO -> 80-C0603X474J4RAUTO; Mouser Price/Stock https://www.mouser.co.uk/ProductDetail/KEMET/C0603C104K4NAC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 -> https://www.mouser.co.uk/ProductDetail/KEMET/C0603X474J4RAC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
- C35: value 47μF -> 0.47μF; footprint GRT32ER60J107ME13L -> PULSE_Library:C0603; Height 2.7 -> 0.87; Manufacturer_Name Murata Electronics -> KEMET; Manufacturer_Part_Number GRT32EC81C476KE13L -> C0603X474J4RACAUTO; Mouser Part Number 81-GRT32EC81C476KE3L -> 80-C0603X474J4RAUTO; Mouser Price/Stock https://www.mouser.co.uk/ProductDetail/Murata-Electronics/G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 -> https://www.mouser.co.uk/ProductDetail/KEMET/C0603X474J4RAC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
- C37, C41: value 1μF -> 4.7μF; footprint C0603 -> C0805; Height 0.87 -> 1.1; Manufacturer_Part_Number C0603X105K4RACAUTO -> C0805C475K4RACAUTO; Mouser Part Number 80-C0603X105K4RAUTO -> 80-C0805C475K4RAUTO; Mouser Price/Stock https://www.mouser.com/Search/Refine.aspx?Keyword=80-C0603X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 -> https://www.mouser.co.uk/ProductDetail/KEMET/C0805C475K4RAC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
- C39: value 47μF -> 4.7μF; footprint GRT32ER60J107ME13L -> C0805; Height 2.7 -> 1.1; Manufacturer_Name Murata Electronics -> KEMET; Manufacturer_Part_Number GRT32EC81C476KE13L -> C0805C475K4RACAUTO; Mouser Part Number 81-GRT32EC81C476KE3L -> 80-C0805C475K4RAUTO; Mouser Price/Stock https://www.mouser.co.uk/ProductDetail/Murata-Electronics/G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 -> https://www.mouser.co.uk/ProductDetail/KEMET/C0805C475K4RAC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
- C40: value 0.1μF -> 4.7μF; footprint C0603 -> C0805; Height 0.87 -> 1.1; Manufacturer_Part_Number C0603C104K4NACAUTO -> C0805C475K4RACAUTO; Mouser Part Number 80-C0603C104K4NAUTO -> 80-C0805C475K4RAUTO; Mouser Price/Stock https://www.mouser.co.uk/ProductDetail/KEMET/C0603C104K4NAC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 -> https://www.mouser.co.uk/ProductDetail/KEMET/C0805C475K4RAC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
- C42: footprint CAPC2012X145N -> PULSE_Library:CAPC2012X145N
- C43: value 0.47μF -> 10μF; footprint C0603 -> PULSE_Library:CAPC2012X145N; Height 0.87 -> 1.45; Manufacturer_Name KEMET -> YAGEO; Manufacturer_Part_Number C0603X474J4RACAUTO -> CC0805KKX7R7BB106; Mouser Part Number 80-C0603X474J4RAUTO -> 603-CC0805KKX77BB106; Mouser Price/Stock https://www.mouser.co.uk/ProductDetail/KEMET/C0603X474J4RAC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 -> https://www.mouser.co.uk/ProductDetail/YAGEO/CC0805KKX7R7BB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
- IC22: renamed from IC24; footprint SOIC127P600X175-8N -> PULSE_Library:SOIC127P600X175-8N
- IC26: renamed from IC?; footprint SOIC127P600X175-8N -> PULSE_Library:SOIC127P600X175-8N
- IC8, IC9: renamed from IC?; footprint SOP50P490X110-10N -> PULSE_Library:SOP50P490X110-10N
- L3, L4, L5: footprint INDPM4440X200N -> PULSE_Library:INDPM4440X200N
- L6: renamed from L1; footprint INDPM4440X200N -> PULSE_Library:INDPM4440X200N
- R11: value 2mΩ -> 2.2MΩ; Manufacturer_Name ROHM Semiconductor -> Susumu; Manufacturer_Part_Number PMR18EZPFV2L00 -> RG3216P-2204-B-T1; Mouser Part Number 755-PMR18EZPFV2L00 -> 754-RG3216P-2204B-T1; Mouser Price/Stock https://www.mouser.co.uk/ProductDetail/ROHM-Semiconductor/P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 -> https://www.mouser.ch/ProductDetail/Susumu/RG3216P-2204-B-T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
- R12, R20, R22: value 2.2MΩ -> 305KΩ; footprint RESC3216X59N -> Resistor_SMD:R_0603_1608Metric; Height 0.59 -> 0.55; Manufacturer_Name Susumu -> KOA Speer; Manufacturer_Part_Number RG3216P-2204-B-T1 -> RN73H1JTTD3053B25; Mouser Part Number 754-RG3216P-2204B-T1 -> 660-RN73H1JTD3053B25; Mouser Price/Stock https://www.mouser.ch/ProductDetail/Susumu/RG3216P-2204-B-T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 -> https://www.mouser.ch/ProductDetail/KOA-Speer/RN73H1JTTD305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
- R14, R24: value 6.12KΩ -> 305KΩ; Manufacturer_Part_Number RN73H1JTTD6121B25 -> RN73H1JTTD3053B25; Mouser Part Number 660-RN73H1JTD6121B25 -> 660-RN73H1JTD3053B25; Mouser Price/Stock https://www.mouser.ch/ProductDetail/KOA-Speer/RN73H1JTTD612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 -> https://www.mouser.ch/ProductDetail/KOA-Speer/RN73H1JTTD305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
- R18, R26: value 583KΩ -> 305KΩ; footprint Resistor_SMD:R_0805_2012Metric_Pad1.20x1.40mm_HandSolder -> Resistor_SMD:R_0603_1608Metric; Manufacturer_Part_Number RN73H2ATTD5833B25 -> RN73H1JTTD3053B25; Mouser Part Number 660-RN73H2ATD5833B25 -> 660-RN73H1JTD3053B25; Mouser Price/Stock https://www.mouser.ch/ProductDetail/KOA-Speer/RN73H2ATTD583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 -> https://www.mouser.ch/ProductDetail/KOA-Speer/RN73H1JTTD305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
- R19, R9: value 6.12KΩ -> 2.2MΩ; footprint Resistor_SMD:R_0603_1608Metric -> RESC3216X59N; Height 0.55 -> 0.59; Manufacturer_Name KOA Speer -> Susumu; Manufacturer_Part_Number RN73H1JTTD6121B25 -> RG3216P-2204-B-T1; Mouser Part Number 660-RN73H1JTD6121B25 -> 754-RG3216P-2204B-T1; Mouser Price/Stock https://www.mouser.ch/ProductDetail/KOA-Speer/RN73H1JTTD612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 -> https://www.mouser.ch/ProductDetail/Susumu/RG3216P-2204-B-T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
- R21: value 305KΩ -> 2.2MΩ; footprint Resistor_SMD:R_0603_1608Metric -> RESC3216X59N; Height 0.55 -> 0.59; Manufacturer_Name KOA Speer -> Susumu; Manufacturer_Part_Number RN73H1JTTD3053B25 -> RG3216P-2204-B-T1; Mouser Part Number 660-RN73H1JTD3053B25 -> 754-RG3216P-2204B-T1; Mouser Price/Stock https://www.mouser.ch/ProductDetail/KOA-Speer/RN73H1JTTD305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 -> https://www.mouser.ch/ProductDetail/Susumu/RG3216P-2204-B-T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
- R23, R25, R27: value 583KΩ -> 2.2MΩ; footprint Resistor_SMD:R_0805_2012Metric_Pad1.20x1.40mm_HandSolder -> RESC3216X59N; Height 0.55 -> 0.59; Manufacturer_Name KOA Speer -> Susumu; Manufacturer_Part_Number RN73H2ATTD5833B25 -> RG3216P-2204-B-T1; Mouser Part Number 660-RN73H2ATD5833B25 -> 754-RG3216P-2204B-T1; Mouser Price/Stock https://www.mouser.ch/ProductDetail/KOA-Speer/RN73H2ATTD583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 -> https://www.mouser.ch/ProductDetail/Susumu/RG3216P-2204-B-T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
- R28: value 22.3KΩ -> 305KΩ; footprint Resistor_SMD:R_0805_2012Metric_Pad1.20x1.40mm_HandSolder -> Resistor_SMD:R_0603_1608Metric; Manufacturer_Part_Number RN73H2ATTD2232B25 -> RN73H1JTTD3053B25; Mouser Part Number 660-RN73H2ATD2232B25 -> 660-RN73H1JTD3053B25; Mouser Price/Stock https://www.mouser.ch/ProductDetail/KOA-Speer/RN73H2ATTD223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 -> https://www.mouser.ch/ProductDetail/KOA-Speer/RN73H1JTTD305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
- R29: value 31.2KΩ -> 6.12KΩ; Manufacturer_Part_Number RN73H1JTTD3122B25 -> RN73H1JTTD6121B25; Mouser Part Number 660-RN73H1JTD3122B25 -> 660-RN73H1JTD6121B25; Mouser Price/Stock https://www.mouser.ch/ProductDetail/KOA-Speer/RN73H1JTTD312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 -> https://www.mouser.ch/ProductDetail/KOA-Speer/RN73H1JTTD612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
- R3, R6, R7, R8: renamed from R?; footprint RESC1608X55N -> PULSE_Library:RESC1608X55N
- R30, R32: value 264KΩ -> 6.12KΩ; footprint Resistor_SMD:R_0805_2012Metric_Pad1.20x1.40mm_HandSolder -> Resistor_SMD:R_0603_1608Metric; Manufacturer_Part_Number RN73H2ATTD2643B25 -> RN73H1JTTD6121B25; Mouser Part Number 660-RN73H2ATD2643B25 -> 660-RN73H1JTD6121B25; Mouser Price/Stock https://www.mouser.ch/ProductDetail/KOA-Speer/RN73H2ATTD264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 -> https://www.mouser.ch/ProductDetail/KOA-Speer/RN73H1JTTD612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
- R31, R33: value 20.8KΩ -> 6.12KΩ; footprint Resistor_SMD:R_0805_2012Metric_Pad1.20x1.40mm_HandSolder -> Resistor_SMD:R_0603_1608Metric; Manufacturer_Part_Number RN73H2ATTD2082B25 -> RN73H1JTTD6121B25; Mouser Part Number 660-RN73H2ATD2082B25 -> 660-RN73H1JTD6121B25; Mouser Price/Stock https://www.mouser.ch/ProductDetail/KOA-Speer/RN73H2ATTD208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 -> https://www.mouser.ch/ProductDetail/KOA-Speer/RN73H1JTTD612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
- R35: value 22.3KΩ -> 2mΩ; footprint Resistor_SMD:R_0805_2012Metric_Pad1.20x1.40mm_HandSolder -> RESC3216X59N; Height 0.55 -> 0.59; Manufacturer_Name KOA Speer -> ROHM Semiconductor; Manufacturer_Part_Number RN73H2ATTD2232B25 -> PMR18EZPFV2L00; Mouser Part Number 660-RN73H2ATD2232B25 -> 755-PMR18EZPFV2L00; Mouser Price/Stock https://www.mouser.ch/ProductDetail/KOA-Speer/RN73H2ATTD223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 -> https://www.mouser.co.uk/ProductDetail/ROHM-Semiconductor/P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
- R5: value 2.2MΩ -> 1.38KΩ; footprint RESC3216X59N -> Resistor_SMD:R_0603_1608Metric; Manufacturer_Name Susumu -> Vishay / Thin Film; Manufacturer_Part_Number RG3216P-2204-B-T1 -> PTN0603E1381BBTS; Mouser Part Number 754-RG3216P-2204B-T1 -> 71-PTN0603E1381BBTS; Mouser Price/Stock https://www.mouser.ch/ProductDetail/Susumu/RG3216P-2204-B-T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 -> https://www.mouser.ch/ProductDetail/Vishay-Thin-Film/PTN060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
- gave numbers to parts that had none: 13
- renumbered C27 to C38, IC4 to IC16
Connections:
- net EN_3.3V_2 is gone; now on net EN: IC16.13 (EN)
- net UHF_Antenna_deploy is gone; now on net GND: C37.1
- net GND: now also C34.2, C36.2, C38.1, C39.1, C40.1, C41.1, C42.1, C43.1, R12.2, R20.2, R22.2, R28.2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; no longer C16.2, C17.2, C18.2, C26.2, C28.2, C38.2, C39.2, C41.2, C42.2, C43.2, D11.1 (A1), D12.1 (A1)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
- net at R31.1: now also IC14.10 (SETI); no longer R30.2
- net at IC12.10 (SETI): now also R29.1
- net at C19.2: now also C17.1, C28.2, D12.1 (A1), IC11.3 (EN), IC11.6 (ANODE), IC4.6 (OUT_1), IC4.7 (OUT_2), Q5.2 (S); no longer L3.2
- net at IC26.3 (VCC): now also C68.1; no longer C41.1
- net at R15.2, R16.1: now also IC15.8 (OVLO)
- net at R10.1: now also IC12.8 (OVLO), R9.2; no longer R13.2
- net at R9.1: now also C32.1, IC12.6 (IN_1), IC12.7 (IN_2), R19.1; no longer IC16.10 (SETI)
- net at IC22.2 (BOOT), IC22.4 (VOUT/FB): now also C57.1; no longer C30.1
- net at R17.2: now also IC16.8 (OVLO), R18.1; no longer R23.1
- net at R24.1: now also R23.2, IC14.9 (UVLO)
- net at C31.1: now also IC11.4 (CATHODE), Q5.3 (D); no longer C32.1
- net at R21.1: now also C33.1, R11.1, IC13.6 (IN_1), IC13.7 (IN_2); no longer R20.2
- net at C34.1: now also R13.1, R23.1, IC14.6 (IN_1), IC14.7 (IN_2)
- net at L5.2: now also C70.2, IC25.1 (SW); no longer C34.2
- net at C19.1: now also C17.2, D12.2 (A2), IC11.2 (GND)
- net at IC22.7 (VIN): now also C65.1
- net at IC22.8 (PGND): now also C65.2, L1.2; no longer L4.2
- net at IC12.9 (UVLO): now also R19.2, R20.1; no longer R27.1
- net at R33.1: now also IC16.10 (SETI); no longer R32.2
- net at C18.1: now also C16.2, D11.2 (A2), IC10.2 (GND)
- net at C37.2: now also C42.2, IC12.14 (OUT_1), IC12.15 (OUT_2), C47.2, D13.1 (A1), IC17.3 (EN), IC17.6 (ANODE), Q6.2 (S); no longer R35.2
- net at C11.1: now also IC4.1 (IN_1), IC4.2 (IN_2), R2.2
- net at L6.2: now also IC26.1 (SW), C71.2
- net at IC26.2 (BOOT): now also C71.1; no longer C40.1
- net at C40.2: now also C45.2, C50.2, D16.1 (A1), IC15.14 (OUT_1), IC15.15 (OUT_2), IC20.3 (EN), IC20.6 (ANODE), Q9.2 (S); no longer IC26.1 (SW)
- net FLAG: now reaches IC12.12 (~{FLAG})
- net FLAG: now also IC16.12 (~{FLAG}), IC13.12 (~{FLAG}), IC14.12 (~{FLAG}), IC15.12 (~{FLAG})
- net at R14.1: now also R13.2, IC14.8 (OVLO)
- net at R25.1: now also C35.1, R15.1, IC15.6 (IN_1), IC15.7 (IN_2)
- net at IC16.14 (OUT_1), IC16.15 (OUT_2): now also C41.2, C46.2, C51.2, D17.1 (A1), IC21.3 (EN), IC21.6 (ANODE), Q10.2 (S); no longer C10.1, C28.1
- net at IC22.6 (AGND): now also C62.1
- net +3.3V: no longer names the net of C24.1, IC9.2 (A0), IC9.6 (VS), R3.2, R7.2
- net +3.3V: no longer C23.1, IC8.6 (VS), R6.2, R8.2
- net 3.3V_1: no longer names the net of IC8.9 (IN-)
- net 3.3V_1: now also IC8.8 (VBUS); no longer R11.1
- removed net 3.3V_1+: C39.1, IC26.4 (VOUT/FB), IC8.10 (IN+), IC8.8 (VBUS), R11.2
- net 3.3V_2: no longer names the net of L6.1
- net 3.3V_2: now also IC26.4 (VOUT/FB), R35.2, C76.1
- net 3.3V_3: no longer names the net of L3.1
- removed net 5V_1+: IC22.5 (EN/CLKIN), IC9.10 (IN+), IC9.8 (VBUS), L4.1, R34.2
- net EN_3.3V_1 renamed EN
- removed net V_bat_in: C13.2, C14.2, C15.2, C16.1, C20.2, C21.2, C22.2, C26.1, C43.1, D10.1 (A1), D11.2 (A2), D12.2 (A2)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
- new net: IC3.8 (~{FAULT}), R1.1
- new net: C10.1, IC3.1 (IN_1), IC3.2 (IN_2), R1.2
- new net: C52.1, IC17.4 (CATHODE), Q6.3 (D)
- new net: IC17.5 (GATE), Q6.1 (G)
- new net: IC15.9 (UVLO), R25.2, R26.1
- new net: C50.1, IC20.1 (VCAP)
- new net: C48.1, IC18.1 (VCAP)
- new net: C38.2, C43.2, C48.2, D14.1 (A1), IC13.14 (OUT_1), IC13.15 (OUT_2), IC18.3 (EN), IC18.6 (ANODE), Q7.2 (S)
- new net: C23.1, IC8.6 (VS), R6.2, R8.2
- new net: C15.2, C22.2, D10.1 (A1), IC7.3 (EN), IC7.6 (ANODE), Q3.2 (S)
- new net: IC4.5 (SET), R5.1
- new net: C70.1, IC25.2 (BOOT)
- new net: IC21.5 (GATE), Q10.1 (G)
- new net: C56.1, IC21.4 (CATHODE), Q10.3 (D)
- new net: C66.1, IC25.3 (VCC)
- new net: C60.1, IC25.5 (EN/CLKIN), IC25.7 (VIN)
- new net: C67.2, IC23.8 (PGND), L3.2
- new net: IC10.5 (GATE), Q4.1 (G)
- new net: C16.1, C18.2, C26.2, D11.1 (A1), IC10.3 (EN), IC10.6 (ANODE), IC3.6 (OUT_1), IC3.7 (OUT_2), Q4.2 (S)
- new net: C30.1, IC10.4 (CATHODE), Q4.3 (D)
- new net: C26.1, IC10.1 (VCAP)
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Other:
- note removed: "OV : 10 V UV : 6 V ILIM : 1 A"
- note removed: "OV : 10 V UV : 6 V ILIM : 4 A"
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
Commit message: changed mcu power suppl
Parts:
- renumbered C10 to C1, C20 to C10, C21 to C11, C22 to C12, C23 to C13, C24 to C14, C25 to C15, C26 to C16, C27 to C17, C28 to C18, C29 to C19, C11 to C2, C30 to C20, C31 to C21, C32 to C22, C33 to C23, C34 to C24, C35 to C25, C36 to C26, C37 to C27, C38 to C28, C39 to C29, C13 to C3, C40 to C30, C41 to C31, C42 to C32, C43 to C33, C44 to C34, C45 to C35, C46 to C36, C47 to C37, C48 to C38, C49 to C39, C14 to C4, C50 to C40, C51 to C41, C52 to C42, C53 to C43, C54 to C44, C55 to C45, C56 to C46, C57 to C47, C58 to C48, C59 to C49, C15 to C5, C60 to C50, C61 to C51, C62 to C52, C63 to C53, C64 to C54, C65 to C55, C66 to C56, C67 to C57, C68 to C58, C69 to C59, C16 to C6, C70 to C60, C71 to C61, C72 to C62, C73 to C63, C74 to C64, C75 to C65, C76 to C66, C17 to C7, C18 to C8, C19 to C9, D8 to D1, D17 to D10, D9 to D2, D10 to D3, D11 to D4, D12 to D5, D13 to D6, D14 to D7, D15 to D8, D16 to D9, IC11 to IC10, IC12 to IC11, IC13 to IC12, IC14 to IC13, IC15 to IC14, IC16 to IC15, IC17 to IC16, IC18 to IC17, IC19 to IC18, IC20 to IC19, IC3 to IC2, IC21 to IC20, IC22 to IC21, IC23 to IC22, IC24 to IC23, IC25 to IC24, IC26 to IC25, IC4 to IC3, IC5 to IC4, IC6 to IC5, IC7 to IC6, IC8 to IC7, IC9 to IC8, IC10 to IC9, L3 to L2, L4 to L3, L5 to L4, L6 to L5
