File: PULSE_ENG.kicad_sch (KiCad schematic)
At the start: 15 parts, among them IC27 ADM3071EARZ, J1 TC2030-MCP, J2 G125-FV10805F3-1AB1ABP, J3 G125-FV10805F3-1AB1ABP, J4 G125-FV10805F3-1AB1ABP, J5 TW-08-07-G-D-375-188, J6 G125-FV10805F3-1AB1ABP, J7 12401832E402A, U1 ATSAMD21J17D-M

Commit message: Adjusting footprints of components
Other:
- moved on the sheet: H1, H2, J1, J5, J7, U1

Commit message: Big final PCU PCB design
Parts:
- added J10: Screw_Terminal_01x01, TerminalBlock_Phoenix:TerminalBlock_Phoenix_MKDS-1,5-2-5.08_1x02_P5.08mm_Horizontal, symbol Connector:Screw_Terminal_01x01
- added J8: Screw_Terminal_01x04, TerminalBlock_Phoenix:TerminalBlock_Phoenix_MKDS-1,5-4-5.08_1x04_P5.08mm_Horizontal, symbol Connector:Screw_Terminal_01x04
- added J9: Screw_Terminal_01x06, TerminalBlock_Phoenix:TerminalBlock_Phoenix_MKDS-1,5-6-5.08_1x06_P5.08mm_Horizontal, symbol Connector:Screw_Terminal_01x06
Connections:
- net BAT_OVP_FLAG: now also U1.41 (PA20)
- net Battery_protection_and_sensing/P_SYS_Protected: now also J10.1 (Pin_1)
- net GND: now also U1.65 (EP), J8.1 (Pin_1), J9.1 (Pin_1), J9.2 (Pin_2); no longer U1.22 (GND), U1.33 (GND), U1.47 (GND), U1.54 (GND)
- net HEATER_SWITCH: now also U1.17 (PA08), J9.6 (Pin_6)
- net I_BAT_ANA: now also U1.10 (PB07)
- net I_PANNEL_ANA: now also U1.11 (PB08)
- net MCU_BAT_EFUSE_EN: now also U1.35 (PA16)
- net MCU_PANNEL_EFUSE_EN: now also U1.36 (PA17)
- net PANNEL_OVP_FLAG: now also U1.42 (PA21)
- net PAN_EFUSE_FLT: now also U1.45 (PA24)
- net PAN_EFUSE_IMON: now also U1.13 (PA04)
- net PAN_EFUSE_PGOOD: now also U1.46 (PA25)
- net POWER_SWITCH: now also U1.18 (PA09), J9.5 (Pin_5)
- net UART1_RX: now also U1.20 (PA11); no longer U1.14 (PA05)
- net UART1_TX: now also U1.19 (PA10); no longer U1.13 (PA04)
- net VBAT_SENSE: now also U1.6 (PB05)
- net VPANNEL_SENSE: now also U1.9 (PB06)
- net Vbat: now also J9.3 (Pin_3), J9.4 (Pin_4)
- net VCHG_RAIL_SENSE: now reaches U1.12 (PB09)
- net GAN_PWM_H: now reaches U1.25 (PB12)
- net GAN_PWM_L: now reaches U1.26 (PB13)
- net BAT_EFUSE_FLT: now reaches U1.37 (PA18)
- net BAT_EFUSE_PGOOD: now reaches U1.38 (PA19)
- net SDA2: now reaches U1.43 (PA22)
- net SCL2: now reaches U1.44 (PA23)
- net BAT_EFUSE_IMON: now reaches U1.5 (PB04)
- new net: U1.22 (GND), U1.33 (GND), U1.47 (GND), U1.54 (GND)
- new net TEST_3V_PDU: J8.2 (Pin_2)
- new net TEST_5V_PDU: J8.3 (Pin_3)
- new net TEST_Pin_SA: J8.4 (Pin_4)
Other:
- sheet Battery_protection_and_sensing ports: added none; removed BAT_HS, BAT_PS, GND
- sheet PCU_Control ports: added VBAT, VCHG_RAIL_SENSE; removed P_SYS_Protected
- sheet PCU_Converter ports: added GROUND; removed gnd
- note added: "TEST CONNECTOR: PWR BATTERY"
- note added: "TEST CONNECTOR: PWR INPUT"
- moved on the sheet: J1

Commit message: Modofications asked and BOM
Parts:
- J10: Mouser Part Number (none) -> 651-1723289; Mouser link (none) -> https://www.mouser.ch/ProductDetail/Phoenix-Contact/1723289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
- J8: Mouser Part Number (none) -> 651-1701144; Mouser link (none) -> https://www.mouser.ch/ProductDetail/Phoenix-Contact/1701144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
- J9: Mouser Part Number (none) -> 651-1730162; Mouser link (none) -> https://www.mouser.ch/ProductDetail/Phoenix-Contact/1730162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
Changed lines of the file:
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@@
+			)
+		)
+		(property "Mouser Part Number" "651-1730162"
+			(at 91.44 232.41 0)
+			(effects
+				(font
+					(size 1.27 1.27)
+				)
+				(hide yes)
+			)
+		)
+		(property "Mouser link" "https://www.mouser.ch/ProductDetail/Phoenix-Contact/1730162?qs=Hp4IEBVVqKI6vRU8VM9TyQ%3D%3D"
+			(at 91.44 232.41 0)
+			(effects
+				(font
+					(size 1.27 1.27)
+				)
+				(hide yes)
 			)
 		)
@@
 			)
 		)
+		(property "Mouser Part Number" "651-1723289"
+			(at 368.3 299.72 0)
+			(effects
+				(font
+					(size 1.27 1.27)
+				)
+				(hide yes)
+			)
+		)
+		(property "Mouser link" "https://www.mouser.ch/ProductDetail/Phoenix-Contact/1723289?qs=ChwaSN6Xm48Jqit%252BJi21%2Fw%3D%3D"
+			(at 368.3 299.72 0)
+			(effects
+				(font
+					(size 1.27 1.27)
+				)
+				(hide yes)
+			)
+		)
 		(pin "1"
 		)
@@
 			(at 49.53 233.68 0)
 			(effects
+				(font
+					(size 1.27 1.27)
+				)
+				(hide yes)
+			)
+		)
+		(property "Mouser Part Number" "651-1701144"
+			(at 49.53 233.68 0)
+			(effects
+				(font
+					(size 1.27 1.27)
+				)
+				(hide yes)
+			)
+		)
+		(property "Mouser link" "https://www.mouser.ch/ProductDetail/Phoenix-Contact/1701144?qs=2WS7V4AoKFp2%2F3%2FlSacg6Q%3D%3D"
+			(at 49.53 233.68 0)
+			(effects

Commit message: changed mcu power suppl
Parts:
- renumbered IC27 to IC1, J2 to J1, J1 to J10, J4 to J2, J6 to J4, J8 to J5, J9 to J6, J10 to J8, J5 to J9
Connections:
- net GNDANA is gone; now on net GND: U1.7 (GNDANA)
- net VDDANA is gone; now on net 3V3: U1.8 (VDDANA)
- net VDDIN is gone; now on net 3V3: U1.56 (VDDIN)
- net VDDIO is gone; now on net 3V3: U1.21 (VDDIO)
- net 3V3: now also U1.34 (VDDIO), U1.48 (VDDIO)
- net GND: now also U1.22 (GND), U1.33 (GND), U1.47 (GND), U1.54 (GND)
Other:
- sheet EPS_Power_Supply ports: added none; removed GNDANA, VDDANA, VDDIN, VDDIO
