File: PULSE_ENG.kicad_pcb (KiCad board)
At the start: 4 copper layers, 146.7 x 93.9 mm, 155 parts, among them IC26 TPS7B8750QDDARQ1, IC27 TPS7B8733QDDARQ1, IC28 INA226AIDGSR, IC29 TPS25940ARVCR, IC30 INA226AIDGSR, IC31 TPS25940ARVCR, J10 TC2030-MCP, J11 Screw_Terminal_01x04, J5 Screw_Terminal_01x04, J6 Screw_Terminal_01x06, J8 Screw_Terminal_01x01, U1 ATSAMD21J17D-M, U2 EPC2152, U3 LM139ADRG4, U4 LT6108IMS8-1-TRPBF, U5 LT6108IMS8-1-TRPBF, Y1 AMDLA4020S-220MT

Commit message: changes
Parts:
- removed MH1, MH2, MH3, MH4: MountingHole, MountingHole:MountingHole_3.2mm_M3
- D16, D17: footprint Diode_THT:D_DO-35_SOD27_P7.62mm_Horizontal -> PULSE_Library:SOD3716X145N
- moved R_BYPASS10 203.7 mm to (47.3, 122.2), turned to 180 degrees
- moved R_BYPASS9 188.1 mm to (52.9, 102.7), turned to 180 degrees
- moved D11 181.1 mm to (51.8, 132.4), turned to 180 degrees
- moved D15 174.4 mm to (60.7, 145.3), turned to 180 degrees
- moved D17 168.0 mm to (66.7, 142.2), turned to 90 degrees
- moved D14 167.1 mm to (66.6, 138.3), turned to 90 degrees
- moved D13 164.0 mm to (74.6, 144.6), turned to 180 degrees
- moved D16 159.0 mm to (77.8, 141.1), turned to 90 degrees
- moved D12 158.9 mm to (77.6, 136.9), turned to 90 degrees
- moved L6 145.6 mm to (95.2, 70.7)
- moved C77 79.2 mm to (147.0, 80.3), turned to 180 degrees
- moved C69 69.9 mm to (144.3, 73.3), turned to 180 degrees
- moved C67 62.7 mm to (151.2, 66.0), turned to 90 degrees
- moved C70 60.8 mm to (152.7, 66.7), turned to 90 degrees
- moved C68 58.4 mm to (158.4, 81.0)
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Routing:
- net GND: track 241.6 -> 274.8 mm, vias 43 -> 47
- net (no net): track 93.2 -> 87.7 mm
- net Net-(D12-K): track 0.00 -> 1.89 mm
- net Net-(D14-K): track 0.00 -> 1.57 mm
- net /PAN_EFUSE_IMON: track 137.6 -> 136.1 mm
- net /BAT_EFUSE_IMON: track 135.7 -> 136.9 mm
- net /3V3: track 543.7 -> 545.0 mm, vias 12 -> 13
- net /I_BAT_ANA: track 100.6 -> 99.5 mm
- net /I_PANNEL_ANA: track 95.8 -> 94.8 mm
