File: PULSE_ENG.kicad_pcb (KiCad board)
At the start: 4 copper layers, 26 parts, among them IC1 TPS7B8733QDDARQ1, IC2 TPS7B8750QDDARQ1, U1 ATSAMD21J17D-M, U4 EPC2152

Commit message: Tom version
Parts:
- removed C1, C4, C5: 100nF, Capacitor_SMD:C_0603_1608Metric_Pad1.08x0.95mm_HandSolder
- removed C10: MBAST105SB7104KFNA01, PULSE_Library:CAPC1005X55N
- removed C2, C3: 10uF, Capacitor_SMD:C_0603_1608Metric_Pad1.08x0.95mm_HandSolder
- removed C6: 1uF, Capacitor_SMD:C_0603_1608Metric_Pad1.08x0.95mm_HandSolder
- removed D1, D2, D3, D4, D5, D6, D7: 1N4148WT, Diode_SMD:D_SOD-523
- removed IC1: TPS7B8733QDDARQ1, PULSE_Library:DDA0008J-IPC_B
- removed IC2: TPS7B8750QDDARQ1, PULSE_Library:DDA0008J-IPC_B
- removed L1: 78404084470, PULSE_Library:78404084470
- removed MH1, MH2, MH3, MH4: MountingHole, MountingHole:MountingHole_3.2mm_M3
- removed U1: ATSAMD21J17D-M, Package_DFN_QFN:QFN-64-1EP_9x9mm_P0.5mm_EP4.7x4.7mm
- added C80: 10nF, PULSE_Library:CAPC2012X145N, F.Cu at (60.5, 42.2)
- added C81: 100nF, Capacitor_SMD:C_0603_1608Metric, F.Cu at (92.7, 68.4)
- added C82: 100nF, Capacitor_SMD:C_0603_1608Metric, F.Cu at (138.3, 111.2)
- added C83: 100nF, Capacitor_SMD:C_0603_1608Metric, F.Cu at (144.9, 115.4)
- added C84: 100nF, Capacitor_SMD:C_0603_1608Metric, F.Cu at (167.7, 112.1)
- added C85: 100nF, Capacitor_SMD:C_0603_1608Metric, F.Cu at (104.4, 98.7)
- added C89: 100nF, Capacitor_SMD:C_0603_1608Metric, F.Cu at (67.4, 64.7)
- added C9: 4.7uF, Capacitor_SMD:C_0201_0603Metric, F.Cu at (92.4, 39.0)
- added C92: 100nF, Capacitor_SMD:C_0603_1608Metric, F.Cu at (66.7, 86.0)
- added C93: 10nF, PULSE_Library:CAPC2012X145N, F.Cu at (60.5, 44.4)
- added D18: 1N4148WT, Diode_SMD:D_SOD-523, F.Cu at (148.7, 67.4)
- added D19: 1N4148WT, Diode_SMD:D_SOD-523, F.Cu at (148.7, 70.4)
- added D20: 1N4148WT, Diode_SMD:D_SOD-523, F.Cu at (148.7, 64.6)
- added D21: 1N4148WT, Diode_SMD:D_SOD-523, F.Cu at (154.1, 78.4)
- added D22: 1N4148WT, Diode_SMD:D_SOD-523, F.Cu at (154.1, 82.0)
- added D23: 1N4148WT, Diode_SMD:D_SOD-523, F.Cu at (154.1, 75.3)
- added IC29: TPS25940ARVCR, PULSE_Library:QFN50P300X400X80-21N, F.Cu at (64.7, 72.5)
- added IC30: TPS25940ARVCR, PULSE_Library:QFN50P300X400X80-21N, F.Cu at (60.6, 93.0)
- added J10: Screw_Terminal_01x01, TerminalBlock_Phoenix:TerminalBlock_Phoenix_MKDS-1,5-2-5.08_1x02_P5.08mm_Horizontal, F.Cu at (52.9, 77.0)
- added J11: Screw_Terminal_01x04, TerminalBlock_Phoenix:TerminalBlock_Phoenix_MKDS-1,5-4-5.08_1x04_P5.08mm_Horizontal, F.Cu at (125.3, 25.1)
- added J12: Screw_Terminal_01x04, TerminalBlock_Phoenix:TerminalBlock_Phoenix_MKDS-1,5-4-5.08_1x04_P5.08mm_Horizontal, F.Cu at (79.5, 51.6)
- added J8: Screw_Terminal_01x04, TerminalBlock_Phoenix:TerminalBlock_Phoenix_MKDS-1,5-4-5.08_1x04_P5.08mm_Horizontal, F.Cu at (46.8, 102.3)
- added J9: Screw_Terminal_01x06, TerminalBlock_Phoenix:TerminalBlock_Phoenix_MKDS-1,5-6-5.08_1x06_P5.08mm_Horizontal, F.Cu at (137.9, 26.6)
- added L**: 78404084470, PULSE_Library:78404084470, F.Cu at (108.5, 46.0)
- added R_BAT_SHUNT1: 20mOhm, Resistor_SMD:R_Shunt_Vishay_WSKW0612, F.Cu at (87.2, 74.9)
- added R_BOT1: 180k, Resistor_SMD:R_0603_1608Metric, F.Cu at (60.3, 40.1)
- added R_BOT2: 180k, Resistor_SMD:R_0603_1608Metric, F.Cu at (141.6, 113.3)
- added R_BOT3: 180k, Resistor_SMD:R_0603_1608Metric, F.Cu at (169.8, 106.9)
- added R_BOT4: 100k, Resistor_SMD:R_0603_1608Metric, F.Cu at (73.0, 99.6)
- added R_BOT5: 180k, Resistor_SMD:R_0603_1608Metric, F.Cu at (135.5, 113.4)
- added R_BOT7: 100k, Resistor_SMD:R_0603_1608Metric, F.Cu at (70.7, 71.1)
- added R_BOT8: 180k, Resistor_SMD:R_0603_1608Metric, F.Cu at (60.5, 47.1)
- added R_BYPASS14: 0, Resistor_SMD:R_0603_1608Metric, F.Cu at (62.7, 77.6)
- added R_BYPASS15: 0, Resistor_SMD:R_0603_1608Metric, F.Cu at (57.4, 97.1)
- added R_BYPASS2: 0, Resistor_SMD:R_0603_1608Metric, F.Cu at (144.0, 69.1)
- added R_BYPASS3: 0, Resistor_SMD:R_0603_1608Metric, F.Cu at (143.9, 71.7)
- added R_BYPASS4: 0, Resistor_SMD:R_0603_1608Metric, F.Cu at (144.1, 66.4)
- added R_BYPASS5: 0, Resistor_SMD:R_0603_1608Metric, F.Cu at (147.0, 79.8)
- added R_BYPASS6: 0, Resistor_SMD:R_0603_1608Metric, F.Cu at (149.1, 83.1)
- added R_BYPASS7: 0, Resistor_SMD:R_0603_1608Metric, F.Cu at (148.2, 76.6)
- added R_FILT10: 402, Resistor_SMD:R_0603_1608Metric, F.Cu at (92.7, 70.1)
- added R_FILT2: 2.61k, Resistor_SMD:R_0603_1608Metric, F.Cu at (96.1, 70.1)
- added R_FILT3: 402, Resistor_SMD:R_0603_1608Metric, F.Cu at (104.4, 100.2)
- added R_FILT4: 2.61k, Resistor_SMD:R_0603_1608Metric, F.Cu at (107.7, 100.2)
- added R_ILIM1: 24k, Resistor_SMD:R_0603_1608Metric, F.Cu at (66.8, 88.9)
- added R_ILIM2: 16.9k, Resistor_SMD:R_0603_1608Metric, F.Cu at (67.3, 67.8)
- added R_IMON1: 4k, Resistor_SMD:R_0603_1608Metric, F.Cu at (66.5, 83.0)
- added R_IMON2: 4k, Resistor_SMD:R_0603_1608Metric, F.Cu at (67.4, 61.8)
- added R_IN1: 100, Resistor_SMD:R_0603_1608Metric, F.Cu at (101.4, 99.5)
- added R_IN2: 100, Resistor_SMD:R_0603_1608Metric, F.Cu at (90.3, 70.1)
- added R_MCU_EN1: 1k, Resistor_SMD:R_0603_1608Metric, F.Cu at (154.0, 67.2)
- added R_MCU_EN2: 1k, Resistor_SMD:R_0603_1608Metric, F.Cu at (160.6, 78.3)
- added R_PANNEL_SHUNT1: 20mOhm, Resistor_SMD:R_Shunt_Vishay_WSKW0612, F.Cu at (98.8, 104.3)
- added R_PD1: 100k, Resistor_SMD:R_0603_1608Metric, F.Cu at (158.4, 71.5)
- added R_PD2: 100k, Resistor_SMD:R_0603_1608Metric, F.Cu at (154.0, 70.5)
- added R_PUP1: 10k, Resistor_SMD:R_0603_1608Metric, F.Cu at (58.1, 71.8)
- added R_PUP2: 10k, Resistor_SMD:R_0603_1608Metric, F.Cu at (144.1, 104.2)
- added R_PUP3: 10k, Resistor_SMD:R_0603_1608Metric, F.Cu at (59.8, 85.2)
- added R_PUP4: 10k, Resistor_SMD:R_0603_1608Metric, F.Cu at (166.1, 99.2)
- added R_PUP5: 10k, Resistor_SMD:R_0603_1608Metric, F.Cu at (55.4, 86.9)
- added R_PUP6: 10k, Resistor_SMD:R_0603_1608Metric, F.Cu at (147.1, 99.2)
- added R_PUP7: 10k, Resistor_SMD:R_0603_1608Metric, F.Cu at (58.0, 68.0)
- added R_TOP1: 680k, Resistor_SMD:R_0603_1608Metric, F.Cu at (52.4, 40.1)
- added R_TOP2: 147k, Resistor_SMD:R_0603_1608Metric, F.Cu at (141.6, 109.3)
- added R_TOP3: 68k, Resistor_SMD:R_0603_1608Metric, F.Cu at (169.8, 99.3)
- added R_TOP4: 681, Resistor_SMD:R_0603_1608Metric, F.Cu at (66.0, 99.6)
- added R_TOP5: 247k, Resistor_SMD:R_0603_1608Metric, F.Cu at (135.4, 109.0)
- added R_TOP7: 681, Resistor_SMD:R_0603_1608Metric, F.Cu at (69.8, 75.6)
- added R_TOP8: 680k, Resistor_SMD:R_0603_1608Metric, F.Cu at (54.7, 47.1)
- added TP11: BAT_EFUSE_EN, TestPoint:TestPoint_Pad_D2.0mm, F.Cu at (167.9, 61.6)
- added TP12: PANNEL_EFUSE_EN, TestPoint:TestPoint_Pad_D2.0mm, F.Cu at (165.2, 79.6)
- added TP27: eFUSE_OVP, TestPoint:TestPoint_Pad_D2.0mm, F.Cu at (70.4, 79.5)
- added TP30: eFuse_EN, TestPoint:TestPoint_Pad_D2.0mm, F.Cu at (67.5, 95.7)
- added TP31: eFuse_OVP, TestPoint:TestPoint_Pad_D2.0mm, F.Cu at (79.5, 96.6)
- added U2: LT6108IMS8-1-TRPBF, PULSE_Library:MSOP-8_MS_LIT, F.Cu at (91.3, 75.0)
- added U3: LM139ADRG4, Package_DIP:CERDIP-14_W7.62mm_SideBrazed_LongPads_Socket, F.Cu at (152.8, 101.7)
- added U5: LT6108IMS8-1-TRPBF, PULSE_Library:MSOP-8_MS_LIT, F.Cu at (103.0, 104.4)
- C7: value MBAST105SB7104KFNA01 -> 100nF; footprint PULSE_Library:CAPC1005X55N -> Capacitor_SMD:C_0201_0603Metric
- C8: value C3216X8L1E106K160AE -> 100nF; footprint PULSE_Library:CAPC3216X180N -> Capacitor_SMD:C_0201_0603Metric
- U4: footprint PULSE_Library:D0122 -> PULSE_Library:VREG_EPC2152ENGRT
- moved C8 80.8 mm to (92.0, 50.0), turned to 0 degrees
- moved U4 69.2 mm to (95.8, 45.6)
- moved C7 66.3 mm to (88.6, 47.7), turned to 180 degrees
- moved C12 54.4 mm to (124.8, 45.6), turned to 180 degrees
Connections:
- C12 pad 2: /PCU_Converter/V_out -> /Vout_BUCK
- C7 pad 1: Net-(C7-Pad1) -> GND
- C7 pad 2: Net-(U4-Vdd12F) -> 12V_1
- C8 pad 1: Net-(C12-Pad1) -> Net-(J11-Pin_3)
- C8 pad 2: /PCU_Converter/V_in -> Net-(C8-Pad2)
- U4 pad 1: Net-(U4-Vdd12F) -> Net-(J11-Pin_3)
- U4 pad 10: Net-(C7-Pad1) -> Net-(C8-Pad2)
- U4 pad 11: Net-(C7-Pad1) -> Net-(C8-Pad2)
- U4 pad 2: /PCU_Converter/V_in_12V -> 12V_1
- U4 pad 3: /PCU_Converter/pwm_H -> /GAN_PWM_H
- U4 pad 4: /PCU_Converter/pwm_L -> /GAN_PWM_L
- U4 pad 5: /PCU_Converter/V_in -> /V_pannel_protected
- U4 pad 6: Net-(C7-Pad1) -> Net-(C8-Pad2)
- U4 pad 7: Net-(C7-Pad1) -> Net-(C8-Pad2)
- U4 pad 8: /PCU_Converter/gnd -> GND
- U4 pad 9: /PCU_Converter/V_in -> /V_pannel_protected
Routing:
- net GND: track 0.00 -> 863.0 mm
- net /3V3: track 0.00 -> 357.3 mm
- net /VBAT_SENSE: track 0.00 -> 236.9 mm
- net /VPANNEL_SENSE: track 0.00 -> 230.0 mm
- net /PANNEL_EFUSE_EN: track 0.00 -> 221.9 mm
- net /Vbat: track 0.00 -> 201.8 mm
- net /V_pannel_protected: track 0.00 -> 166.2 mm
- net /BAT_EFUSE_EN: track 0.00 -> 159.5 mm
- net /Vout_BUCK: track 0.00 -> 124.6 mm
- net /PCU_Control/BAT_OVC: track 0.00 -> 114.5 mm
- net /PCU_Control/PANNEL_OVC: track 0.00 -> 107.5 mm
- net Net-(J11-Pin_3): track 0.00 -> 79.3 mm
- net /MCU_PANNEL_EFUSE_EN: track 0.00 -> 76.0 mm
- net /MCU_BAT_EFUSE_EN: track 0.00 -> 72.7 mm
- net /BAT_OVP_FLAG: track 0.00 -> 71.0 mm
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Other:
- board outline added: 146.7 x 106.9 mm
