File: Control.kicad_sch (KiCad schematic)
At the start: 0 parts

Commit message: Tom version
Parts:
- added C10, C11, C14, C15: 100nF, CAPC1005X55N, symbol PULSE_Library:MBAST105SB7104KFNA01
- added C13: MBAST105SB7104KFNA01, CAPC1005X55N, symbol PULSE_Library:MBAST105SB7104KFNA01
- added C80, C93: 10nF, PULSE_Library:CAPC2012X145N, symbol PULSE_Library:C2012X7R1A106M125AC
- added D18, D19, D20, D21, D22, D23: 1N4148WT, Diode_SMD:D_SOD-523, symbol Diode:1N4148WT
- added R_BOT1, R_BOT2, R_BOT3, R_BOT5, R_BOT8: 180k, Resistor_SMD:R_0603_1608Metric, symbol Device:R
- added R_BYPASS2, R_BYPASS3, R_BYPASS4, R_BYPASS5, R_BYPASS6, R_BYPASS7: 0, Resistor_SMD:R_0603_1608Metric, symbol Device:R
- added R_FILT10, R_FILT3: 402, Resistor_SMD:R_0603_1608Metric, symbol Device:R
- added R_FILT2, R_FILT4: 2.61k, Resistor_SMD:R_0603_1608Metric, symbol Device:R
- added R_IN1, R_IN2: 100, Resistor_SMD:R_0603_1608Metric, symbol Device:R
- added R_MCU_EN1, R_MCU_EN2: 1k, Resistor_SMD:R_0603_1608Metric, symbol Device:R
- added R_PD1, R_PD2: 100k, Resistor_SMD:R_0603_1608Metric, symbol Device:R
- added R_PUP2, R_PUP4, R_PUP6: 10k, Resistor_SMD:R_0603_1608Metric, symbol Device:R
- added R_TOP1, R_TOP8: 680k, Resistor_SMD:R_0603_1608Metric, symbol Device:R
- added R_TOP2: 147k, Resistor_SMD:R_0603_1608Metric, symbol Device:R
- added R_TOP3: 68k, Resistor_SMD:R_0603_1608Metric, symbol Device:R
- added R_TOP5: 247k, Resistor_SMD:R_0603_1608Metric, symbol Device:R
- added R_hyst1, R_hyst2, R_hyst3: 1MOhm, Resistor_SMD:R_0603_1608Metric, symbol Device:R
- added TP1: IBAT_ANA, TestPoint:TestPoint_Pad_D2.0mm, symbol Connector:TestPoint_Probe
- added TP10: VBAT_SENSE, TestPoint:TestPoint_Pad_D2.0mm, symbol Connector:TestPoint_Probe
- added TP11: BAT_EFUSE_EN, TestPoint:TestPoint_Pad_D2.0mm, symbol Connector:TestPoint_Probe
- added TP12: PANNEL_EFUSE_EN, TestPoint:TestPoint_Pad_D2.0mm, symbol Connector:TestPoint_Probe
- added TP13: MCU_BAT_EFUSE_EN, TestPoint:TestPoint_Pad_D2.0mm, symbol Connector:TestPoint_Probe
- added TP14: MCU_PANNEL_EFUSE_EN, TestPoint:TestPoint_Pad_D2.0mm, symbol Connector:TestPoint_Probe
- added TP15: BAT_UVP, TestPoint:TestPoint_Pad_D2.0mm, symbol Connector:TestPoint_Probe
- added TP16: BAT_OVP, TestPoint:TestPoint_Pad_D2.0mm, symbol Connector:TestPoint_Probe
- added TP17: PANNEL_OVP, TestPoint:TestPoint_Pad_D2.0mm, symbol Connector:TestPoint_Probe
- added TP18: BAT_SHUNT_OUT, TestPoint:TestPoint_Pad_D2.0mm, symbol Connector:TestPoint_Probe
- added TP19: BAT_SHUNT_IN, TestPoint:TestPoint_Pad_D2.0mm, symbol Connector:TestPoint_Probe
- added TP20: PANNEL_SHUNT_OUT, TestPoint:TestPoint_Pad_D2.0mm, symbol Connector:TestPoint_Probe
- added TP21: PANNEL_SHUNT_IN, TestPoint:TestPoint_Pad_D2.0mm, symbol Connector:TestPoint_Probe
- added TP3: IPANNEL_ANA, TestPoint:TestPoint_Pad_D2.0mm, symbol Connector:TestPoint_Probe
- added TP8: VPANNEL_SENSE, TestPoint:TestPoint_Pad_D2.0mm, symbol Connector:TestPoint_Probe
- added U2, U5: LT6108IMS8-1-TRPBF, PULSE_Library:MSOP-8_MS_LIT, symbol PULSE_Library:LT6108IMS8-1-TRPBF
- added U3: LM139ADRG4, Package_DIP:CERDIP-14_W7.62mm_SideBrazed_LongPads_Socket, symbol PULSE_Library:LM139ADRG4
Connections:
- new net: R_IN2.1, U2.8 (SENSEHI)
- new net: R_FILT10.1, R_FILT2.2, U2.5 (INC)
- new net: D18.1 (K), R_BYPASS2.2
- new net: D19.1 (K), R_BYPASS3.2
- new net: R_BOT5.2, R_TOP5.1, U3.7 (1IN+)
- new net: D20.1 (K), R_BYPASS4.2
- new net: D23.1 (K), R_BYPASS7.2
- new net: R_BOT3.2, R_TOP3.1, U3.8 (3IN-)
- new net: D22.1 (K), R_BYPASS6.2
- new net: R_IN1.1, U5.8 (SENSEHI)
- new net: R_FILT3.1, R_FILT4.2, U5.5 (INC)
- new net: R_BOT2.2, R_TOP2.1, U3.4 (2IN-)
- new net: D21.1 (K), R_BYPASS5.2
- new net 3.3V: C10.2, R_PUP2.1, R_PUP4.2, R_PUP6.1, R_TOP2.2, R_TOP3.2, R_TOP5.2, U2.2 (EN/*RST), U3.3 (VCC), U5.2 (EN/*RST)
- new net BAT_EFUSE_EN: D18.2 (A), D19.2 (A), D20.2 (A), R_MCU_EN1.1, R_PD2.2, TP11.1
- new net BAT_OVC: R_BYPASS4.1, U2.3 (OUTC)
- new net BAT_OVP_FLAG: R_BYPASS2.1, R_BYPASS5.1, R_PUP2.2, R_hyst3.2, TP16.1, U3.2 (2OUT)
- new net BAT_SHUNT_IN: R_IN2.2, TP19.1, U2.7 (V+)
- new net BAT_SHUNT_OUT: TP18.1, U2.1 (SENSELO)
- new net BAT_UVP_FLAG: R_BYPASS3.1, R_PUP6.2, R_hyst2.2, TP15.1, U3.1 (1OUT)
- new net BUCK_IN: R_TOP1.1
- new net GND: C10.1, C11.1, C13.1, C14.1, C15.1, C80.2, C93.2, R_BOT1.1, R_BOT2.1, R_BOT3.1, R_BOT5.1, R_BOT8.1, R_FILT2.1, R_FILT4.1, R_PD1.1, R_PD2.1, U2.4 (V-), U3.12 (GND), U5.4 (V-)
- new net I_BAT_ANA: C15.2, R_FILT10.2, TP1.1, U2.6 (OUTA)
- new net I_PANNEL_ANA: C14.2, R_FILT3.2, TP3.1, U5.6 (OUTA)
- new net MCU_BAT_EFUSE_EN: R_MCU_EN1.2, TP13.1
- new net MCU_PANNEL_EFUSE_EN: R_MCU_EN2.2, TP14.1
- new net PANNEL_EFUSE_EN: D21.2 (A), D22.2 (A), D23.2 (A), R_MCU_EN2.1, R_PD1.2, TP12.1
- new net PANNEL_OVC: R_BYPASS7.1, U5.3 (OUTC)
- new net PANNEL_OVP_FLAG: R_BYPASS6.1, R_PUP4.1, R_hyst1.2, TP17.1, U3.14 (OUT3)
- new net PANNEL_SHUNT_IN: R_IN1.2, TP21.1, U5.7 (V+)
- new net PANNEL_SHUNT_OUT: TP20.1, U5.1 (SENSELO)
- new net VBAT: R_TOP8.1
- new net VBAT_SENSE: C11.2, C93.1, R_BOT8.2, R_TOP8.2, R_hyst2.1, R_hyst3.1, TP10.1, U3.5 (2IN+), U3.6 (1IN-)
- new net VPANNEL_SENSE: C13.2, C80.1, R_BOT1.2, R_TOP1.2, R_hyst1.1, TP8.1, U3.9 (3IN+)
- no-connect marks 0 -> 3
Other:
- note added: "ENABLE SIGNALS LOGIC"
- note added: "GROUNDING"
- note added: "INPUTS"
- note added: "OUTPUTS"
- note added: "OVERCURRENT HARDWARE CUTOFF"
- note added: "OVERVOLTAGE HARDWARE CUTOFF"
- note added: "VOLTAGE SENSING"
- company: EPFL Spacecraft Team -> (none)
