File: PCU.kicad_sch (KiCad schematic)
At the start: 7 parts, among them U4 EPC2152, Y1 AMDLA4020S-220MT

Commit message: pcb trial
Parts:
- removed C7, C8: 100nF, symbol SamacSys_Parts:C
- removed C9: 4.7uF, symbol SamacSys_Parts:C
- removed L2: 47, symbol SamacSys_Parts:L
- removed Y1: AMDLA4020S-220MT, PULSE_Library:INDPM4440X200N, symbol PULSE_Library:AMDLA4020S-220MT
- added C10, C7: MBAST105SB7104KFNA01, CAPC1005X55N, symbol PULSE_Library:MBAST105SB7104KFNA01
- added C8: C3216X8L1E106K160AE, CAPC3216X180N, symbol PULSE_Library:C3216X8L1E106K160AE
- added L1: 78404084470, 78404084470, symbol PULSE_Library:78404084470
- U4: footprint EPC_FETs:D0122 -> PULSE_Library:D0122
Connections:
- net V_in: now also C8.2
- net V_in_12V: now also C10.2
- net V_out: now also L1.2
- net gnd: now also C10.1
- net at C12.1, U4.12 (Vss): now also C8.1
- net at U4.1 (Vdd12F): now also C7.2
- net at U4.10 (SW), U4.11 (SW), U4.6 (SW)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: now also C7.1, L1.1
Other:
- moved on the sheet: C12

Commit message: Tom version
Parts:
- removed C10: MBAST105SB7104KFNA01, CAPC1005X55N, symbol PULSE_Library:MBAST105SB7104KFNA01
- removed C8: C3216X8L1E106K160AE, CAPC3216X180N, symbol PULSE_Library:C3216X8L1E106K160AE
- added C8: MBAST105SB7104KFNA01, CAPC1005X55N, symbol PULSE_Library:MBAST105SB7104KFNA01
- added C9: 10uF, PULSE_Library:CAPC3216X180N, symbol PULSE_Library:C3216X8L1E106K160AE
- added J11: Screw_Terminal_01x04, TerminalBlock_Phoenix:TerminalBlock_Phoenix_MKDS-1,5-4-5.08_1x04_P5.08mm_Horizontal, symbol Connector:Screw_Terminal_01x04
- added TP2: 12Vin_buck, TestPoint:TestPoint_Pad_D2.0mm, symbol Connector:TestPoint_Probe
- added TP5: PWM_H, TestPoint:TestPoint_Pad_D2.0mm, symbol Connector:TestPoint_Probe
- added TP6: PWM_L, TestPoint:TestPoint_Pad_D2.0mm, symbol Connector:TestPoint_Probe
- added TP7: Buck_out, TestPoint:TestPoint_Pad_D2.0mm, symbol Connector:TestPoint_2Pole
- C12: value C3216X8L1E106K160AE -> 10uF; footprint CAPC3216X180N -> PULSE_Library:CAPC3216X180N
- C7: value MBAST105SB7104KFNA01 -> 100nF
- U4: footprint PULSE_Library:D0122 -> PULSE_Library:VREG_EPC2152ENGRT
Connections:
- net V_in: now also C9.2
- net V_in_12V: now also C7.2, J11.1 (Pin_1), TP2.1
- net V_out: now also J11.2 (Pin_2), TP7.1
- net pwm_H: now also TP5.1
- net pwm_L: now also TP6.1
- net at L1.1, U4.10 (SW), U4.11 (SW)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: now also C8.1; no longer C7.1
- net at U4.1 (Vdd12F): now also C8.2, J11.3 (Pin_3); no longer C7.2
- net at C12.1, U4.12 (Vss): now also C9.1, TP7.2
- net gnd renamed GROUND
- net GROUND: now also C7.1
- new net GND: J11.4 (Pin_4)
Other:
- note added: "pas sure de cette valeur pour C_in"
- company: EPFL Spacecraft Team -> (none)
- moved on the sheet: C12, L1, U4
