File: untitled.kicad_sch (KiCad schematic)
At the start: 22 parts, among them IC28 INA226AIDGSR, IC29 TPS25940ARVCR

Commit message: lastest
Parts:
- removed C_DVDT, C_FILT, C_FILT1: 100nF, symbol Device:C
- removed NT1, NT2: NetTie_2, symbol Device:NetTie_2
- added C86, C88, C89: 100nF, Capacitor_SMD:C_0603_1608Metric, symbol PULSE_Library:C0603X6S0J104M030BC
- added R_BYPASS14: 0, Resistor_SMD:R_0603_1608Metric, symbol Device:R
- added TP24: eFUSE_EN, TestPoint:TestPoint_Pad_D2.0mm, symbol Connector:TestPoint_Probe
- added TP25: Buck_out, TestPoint:TestPoint_Pad_D2.0mm, symbol Connector:TestPoint_Probe
- added TP27: eFUSE_OVP, TestPoint:TestPoint_Pad_D2.0mm, symbol Connector:TestPoint_Probe
- C77: footprint (none) -> Capacitor_SMD:C_0201_0603Metric
- C78: footprint C0603 -> PULSE_Library:C0603
- IC28: footprint SOP50P490X110-10N -> PULSE_Library:SOP50P490X110-10N
- R37, R38: footprint RESC1608X55N -> PULSE_Library:RESC1608X55N
- R_ADD_CONFIG1, R_FILT1, R_PUP1: footprint (none) -> Resistor_SMD:R_0603_1608Metric
- R_ADD_CONFIG4: renamed from R_ADD_CONFIG; footprint (none) -> Resistor_SMD:R_0603_1608Metric
- R_BAT_SHUNT1: renamed from R_BAT_SHUNT; footprint (none) -> Resistor_SMD:R_Shunt_Vishay_WSKW0612
- R_BOT7: renamed from R_BOT; footprint (none) -> Resistor_SMD:R_0603_1608Metric
- R_FILT7: renamed from R_FILT; footprint (none) -> Resistor_SMD:R_0603_1608Metric
- R_ILIM2: renamed from R_ILIM; footprint (none) -> Resistor_SMD:R_0603_1608Metric
- R_IMON2: renamed from R_IMON; footprint (none) -> Resistor_SMD:R_0603_1608Metric
- R_PUP7: renamed from R_PUP; footprint (none) -> Resistor_SMD:R_0603_1608Metric
- R_TOP7: renamed from R_TOP; footprint (none) -> Resistor_SMD:R_0603_1608Metric
Connections:
- net Vbat is gone; now on net BAT_POS: R_BAT_SHUNT1.4
- net BAT_EFUSE_EN: now also TP24.1
- net BUCK_OUT: now also R_BYPASS14.1, TP25.1
- net GND: now also C86.2, C88.2, C89.1
- net P_SYS_Protected: now also R_BYPASS14.2
- net at IC28.8 (VBUS), IC28.9 (IN-), R_FILT1.2: now also C88.1; no longer IC28.10 (IN+)
- net at IC29.18 (DVDT): now also C89.2
- net at R_FILT7.2: now also IC28.10 (IN+), C86.1
- net at IC29.15 (OVP), R_BOT7.1, R_TOP7.2: now also TP27.1
- no-connect marks 1 -> 3
Other:
- moved on the sheet: C77, C78, IC28, IC29, R37, R38, R_ADD_CONFIG1, R_ADD_CONFIG4, R_BAT_SHUNT1, R_BOT7, R_FILT1, R_FILT7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
